Commit message: Fix Ranger's green path display, wall standoff, and missing wheels
Found via actual RViz/Gazebo inspection (not caught by the previous
commit's topic-level-only testing):

- ranger_xarm6.rviz had no Path display for path_topic at all; even
  after adding one, it rendered nothing until Buffer Length: 1 was set
  (confirmed missing by diffing against the old Robotnik rviz config,
  which has it) -- the property tf2_ros/rviz needs to actually draw a
  received nav_msgs/Path, not just accept the message.
- Ranger's Initial Position EE standoff from the wall was ~0.25m
  (x=2.60), further than Theron/Kairos's own ready poses look. Reduced
  to ~0.05m (x=2.80, matching path.yaml's own waypoint x) by
  re-solving the IK target; manipulability improved too (0.80 vs the
  previous 0.37).
- The base's 4 steering + 4 wheel joints have no ros2_control
  interface (by design, base driving is separate follow-up work), so
  nothing published their joint state and RobotModel had no TF for
  them -- they were rendering as entirely absent, not just static.
  Added a state-only ros2_control block (no command interface) so
  joint_state_broadcaster picks them up and they render.

All three verified visually this round via DISPLAY=:1 + PIL
screenshots (docs/initial_position_ik_notes.md has the debugging
trail, including a couple of dead ends before finding Buffer Length).

Co-Authored-By: Claude Sonnet 5 <noreply@anthropic.com>

File: robots/ranger_xarm6.urdf.xacro (robot description, xacro)
@@ -74,4 +74,44 @@
     </gazebo>
   </xacro:if>
+  <!-- State-only ros2_control interface for the base's 4 steering + 4 wheel
+       joints (see ranger_mini_v3.xacro's own header comment: they're left
+       passive, no command interface / drive plugin; driving the base is
+       still separate follow-up work, unchanged by this). Without any
+       ros2_control interface, nothing ever published these joints' state,
+       so robot_state_publisher had no value for them and couldn't compute
+       their TF: RViz's RobotModel display then has no transform for the
+       wheel/steering links and hides them entirely (not just "not moving",
+       genuinely absent). Declaring them here with state_interface only (no
+       command_interface, no new controller) lets gz_ros2_control's
+       GazeboSimSystem report their actual simulated pose, picked up by
+       the same joint_state_broadcaster the arm already uses (it publishes
+       every joint from every claimed hardware interface by default, see
+       config/ros2_controllers.yaml: no 'joints' list there means "all of
+       them"), so the wheels/steering render (static, since nothing drives
+       them yet) instead of disappearing. Real hardware isn't affected:
+       this whole block is gz-sim-only (_is_gz_sim), same as the plugin
+       block above.
+  -->
+  <xacro:if value="${_is_gz_sim}">
+    <ros2_control name="RangerBaseState" type="system">
+      <hardware>
+        <plugin>gz_ros2_control/GazeboSimSystem</plugin>
+      </hardware>
+      <xacro:macro name="_passive_wheel_joint" params="name">
+        <joint name="$(arg prefix)${name}">
+          <state_interface name="position"/>
+          <state_interface name="velocity"/>
+        </joint>
+      </xacro:macro>
+      <xacro:_passive_wheel_joint name="fl_steering_joint"/>
+      <xacro:_passive_wheel_joint name="fl_wheel"/>
+      <xacro:_passive_wheel_joint name="fr_steering_joint"/>
+      <xacro:_passive_wheel_joint name="fr_wheel"/>
+      <xacro:_passive_wheel_joint name="rl_steering_joint"/>
+      <xacro:_passive_wheel_joint name="rl_wheel"/>
+      <xacro:_passive_wheel_joint name="rr_steering_joint"/>
+      <xacro:_passive_wheel_joint name="rr_wheel"/>
+    </ros2_control>
+  </xacro:if>
   <!-- F/T SENSOR (Gazebo simulation only). Assumed present for this
        integration, per instruction: treat sim force/contact behaviour as

Commit message: Reach the path's actual start point; fix a base-height bug in wbc.py
Ranger's Initial Position EE was reaching only z=0.95, well short of
the wall path's actual first waypoint (path.yaml: [2.80, 4.9, 1.3]).
At the original 0.05m arm_base_joint mount, z=1.3 isn't reachable at
any base standoff, including the chassis touching the wall -- so this
moves the base closer (RANGER_INIT_BASE_X 2.35 -> 2.5, chassis still
clears the wall by ~0.10m) and raises the mount to 0.3m (both
ranger_xarm6.urdf.xacro and urdf/ranger_xarm6.urdf).

Re-deriving the IK caught a methodology bug in the previous commit's
numbers (init_joint_positions there landed at world z=1.40, not 1.30,
confirmed against live TF -- a wrong-but-plausible answer the solver's
own success flag didn't catch): roboticstoolbox's
robot.ets(start='arm_base_link', ...) silently includes whatever
arm_mount_xyz is currently on disk rather than excluding it as "start="
suggests, so manually subtracting the mount again double-counted it;
separately, wbc.py's base-transform convention hardcodes world z=0,
so an IK target needs world_z - RANGER_INIT_BASE_Z, not world_z. New
init_joint_positions verified against live Gazebo TF
(robot_a_odom -> robot_a_link_eef reads (2.800, 4.899, 1.300)).

That same base-height convention bug was real in wbc.py itself:
update_robot_state() read tx/ty/yaw from the odom->base_link TF but
never tz, silently assuming the base sits at ground level. True for
Theron/Kairos, false for Ranger (0.15m chassis clearance) -- every
p_ee estimate, and so every path-tracking error computed from it, was
biased low by that much. Fixed by reading and including tz. Also
updated solve_full_qp's Ranger wall-regulation constant (2.35 -> 2.5)
to match the standoff actually verified above.

Checked, but not fixed here: Ranger's wheels have no ros2_control
command interface (no drive plugin wired up, by design -- see
ranger_mini_v3.xacro), so run_trajectory_control()'s base cmd_vel goes
nowhere and odom->base_link never updates live either. That's almost
certainly the dominant reason path tracking fails beyond whatever
fraction of the ~9.8m-wide path falls within the arm's own ~0.7m
reach of wherever the base is parked -- no amount of QP correctness
fixes that without a real drive plugin (sim) or the ranger_ros2 driver
(hardware) actually wired up. Flagged in
docs/initial_position_ik_notes.md rather than worked around.

Co-Authored-By: Claude Sonnet 5 <noreply@anthropic.com>

File: robots/ranger_xarm6.urdf.xacro (robot description, xacro)
@@ -38,9 +38,13 @@
        PLACEHOLDER FT: base -> arm mount transform.
        No physical Ranger Mini 3 + xArm6 hardware access yet, so this offset
-       is NOT measured: it just centers the arm base on top of the chassis
-       deck with a nominal 5cm mounting plate, clear of the collision box.
-       Replace attach_xyz/attach_rpy below once the real mount is measured.
+       is NOT measured. Raised from an original 5cm nominal mounting-plate
+       guess to 0.3m: at 0.05m the arm could not reach the wall path's top
+       waypoint (world z=1.3) at any base standoff from the wall, including
+       the chassis touching it; see docs/initial_position_ik_notes.md for
+       the IK sweep. 0.3m is still a guess (a riser/pedestal, not a thin
+       plate), not a measurement; replace attach_xyz/attach_rpy below once
+       the real mount is measured.
        ==================================================================== -->
-  <xacro:property name="arm_mount_xyz" value="0 0 0.05" />
+  <xacro:property name="arm_mount_xyz" value="0 0 0.3" />
   <xacro:property name="arm_mount_rpy" value="0 0 0" />
   <!-- Base: Ranger Mini 3.0 -->

Commit message: Fix three real bugs blocking Ranger+xArm6 tracking; remove Theron/Kairos support
Three confirmed bugs fixed in wbc.py, found while debugging why FDCC lost
contact and drifted over time on Ranger+xArm6 (none of these are tuning
issues):

1. Base wall-standoff cost regulated the wrong DOF. Ranger spawns at
   yaw=-pi/2 (sideways to the wall, unlike Theron/Kairos), which flips
   which virtual base joint maps to which world axis. Verified
   numerically (perturb each base joint, read the FK delta): q[1] ("v_x")
   moves world -Y (sweep axis), q[2] ("v_y") moves world +X (the actual
   wall-approach axis). The standoff cost was on c[1]; moved to c[2].

2. joint_velocity_damper() called with positional args that don't match
   the installed roboticstoolbox (1.4.3) signature
   (q=None, ps=0.05, pi=0.1, n=None, gain=1.0). Calling it as
   (0.1, 0.9, n_joints) put 0.1 into q (a bare float, not an array),
   raising TypeError the instant it's indexed -- silently swallowed by a
   try/except that zeroed the joint-limit inequality constraint,
   disabling joint-limit avoidance entirely. xArm6's joint2/joint3 have
   far tighter ranges than UR5e and got driven straight into their hard
   limits mid-trajectory without this. Fixed: call by keyword.

3. wbc.py wasn't sim-time-aware. self.get_clock().now() was the wall
   clock, but control_loop()'s ROS timer fires at a rock-solid 100.00Hz
   in wall-clock time regardless of Gazebo's real_time_factor (measured
   live: RTF drops to 0.24-0.5 under QP+physics load, control-loop timing
   unaffected). The trapezoidal trajectory reference was advancing at
   full wall-clock speed while the robot's physics only progressed at
   30-50% of that rate -- an unbounded, ever-growing drift for as long as
   the trajectory ran. This is what "FDCC drifts over time" actually was.
   Fixed by adding use_sim_time: true to wbc.py's launch parameters,
   matching what base_pose_publisher.py already did correctly.

Also tried and reverted: lowering the base-motion QP cost for Ranger's
translation DOFs (kept omega's cost unchanged after an earlier attempt to
lower that too caused unwanted base rotation). Looked like an improvement
in logged error metrics, but visibly worsened base motion in practice, so
reverted to the original uniform penalty.

max_ee_vel/max_ee_accel promoted from hardcoded instance attributes to
declared ROS parameters, so future tuning doesn't need a rebuild.

Removed Theron/Kairos/Robotnik/UR5e support from this branch (standalone
scripts, URDFs, launch args) since this branch is AgileX-only -- that
support remains on main. Kept the RobotType enum / robot_type parameter
dispatch pattern rather than hardcoding to Ranger, since more AgileX
bases (e.g. Scout) + xArm6 are expected on this branch later.

Still open: tangential tracking error (ey/ez) cycles between ~0 and
250-350mm roughly every 25-40s throughout the path. Ruled out simple
gain/speed tuning (tried both raising v_max_traj and lowering
max_ee_vel, neither helped) and ruled out the low-level velocity
controller (isolated step-response test tracks a commanded velocity in
~50ms for both gravity-loaded and light joints). Base motion is
continuous and smooth during the cycle, so it isn't simply "base too
slow to engage" either. Needs correlation against path geometry or live
manipulability data next.

Co-Authored-By: Claude Sonnet 5 <noreply@anthropic.com>

File: robots/ranger_xarm6.urdf.xacro (robot description, xacro)
@@ -44,13 +44,13 @@
        PLACEHOLDER FT: base -> arm mount transform.
        No physical Ranger Mini 3 + xArm6 hardware access yet, so this offset
-       is NOT measured. Raised from an original 5cm nominal mounting-plate
-       guess to 0.3m: at 0.05m the arm could not reach the wall path's top
-       waypoint (world z=1.3) at any base standoff from the wall, including
-       the chassis touching it; see docs/initial_position_ik_notes.md for
-       the IK sweep. 0.3m is still a guess (a riser/pedestal, not a thin
-       plate), not a measurement; replace attach_xyz/attach_rpy below once
-       the real mount is measured.
+       is NOT measured: 0.05m is a nominal thin mounting-plate guess.
+       (A prior revision temporarily raised this to 0.3m, a pedestal-height
+       guess, purely so the arm could reach an artificially high path
+       waypoint; reverted now that the path itself was shifted down to a
+       reasonable height instead: see wbcc_path/path/path.yaml and
+       docs/initial_position_ik_notes.md.) Replace attach_xyz/attach_rpy
+       below once the real mount is measured.
        ==================================================================== -->
-  <xacro:property name="arm_mount_xyz" value="0 0 0.3" />
+  <xacro:property name="arm_mount_xyz" value="0 0 0.05" />
   <xacro:property name="arm_mount_rpy" value="0 0 0" />
   <!-- Base: Ranger Mini 3.0 -->

Commit message: Correct base->arm mount FT via Gazebo visual inspection
The STEP-file-derived mount transform (arm_mount_xyz/arm_mount_rpy in
ranger_xarm6.urdf.xacro, mirrored in urdf/ranger_xarm6.urdf) placed the
arm too high and at the wrong yaw once actually viewed in Gazebo.

Root cause: the mounting-plate height (0.25368m) was measured relative
to the STEP CAD's "Ranger Mini 3.0" node origin, which is not the same
reference point as this package's base_link (base_link sits near the
top of the chassis per ranger_mini_v3.xacro's collision box/visual
mesh, while the STEP node's origin is deeper inside the body). x
(-0.2185) checked out visually and is unaffected.

Corrected z to 0.024m and yaw to 180 degrees by direct visual
inspection in Gazebo. Still provisional pending a real hardware
measurement or confirmation against the ARTC handover note.

Co-Authored-By: Claude Sonnet 5 <noreply@anthropic.com>

File: robots/ranger_xarm6.urdf.xacro (robot description, xacro)
@@ -42,16 +42,25 @@
   <xacro:arg name="robot_ip" default="" />
   <!-- ====================================================================
-       PLACEHOLDER FT: base -> arm mount transform.
-       No physical Ranger Mini 3 + xArm6 hardware access yet, so this offset
-       is NOT measured: 0.05m is a nominal thin mounting-plate guess.
-       (A prior revision temporarily raised this to 0.3m, a pedestal-height
-       guess, purely so the arm could reach an artificially high path
-       waypoint; reverted now that the path itself was shifted down to a
-       reasonable height instead: see wbcc_path/path/path.yaml and
-       docs/initial_position_ik_notes.md.) Replace attach_xyz/attach_rpy
-       below once the real mount is measured.
+       FT: base -> arm mount transform, corrected from Gazebo visual
+       inspection after the STEP-derived heights kept turning out wrong.
+       x=-0.2185 (from the mounting-plate geometry in
+       RM_Version_1.2_production.step) checked out visually. z, however,
+       was wrong at 0.25368 (mount plate height relative to the STEP CAD's
+       "Ranger Mini 3.0" node origin), that STEP node's own origin isn't
+       the same reference point as this package's base_link (base_link
+       sits near the top of the chassis per ranger_mini_v3.xacro's
+       collision box / visual mesh; the STEP node's origin is lower, deeper
+       inside the chassis body), so the two aren't directly comparable
+       without correcting for that offset. z set to 0.024 (24mm) per direct
+       visual correction in Gazebo (arm was floating too high). Yaw set to
+       180 degrees, also per visual correction. Still not a hardware
+       measurement, treat as provisional until the real mount is
+       physically measured or the arm's true orientation is confirmed
+       against the ARTC handover note.
+       Kept numerically in sync with arm_base_joint's origin in
+       urdf/ranger_xarm6.urdf.
        ==================================================================== -->
-  <xacro:property name="arm_mount_xyz" value="0 0 0.05" />
-  <xacro:property name="arm_mount_rpy" value="0 0 0" />
+  <xacro:property name="arm_mount_xyz" value="-0.218500 0.000000 0.024000" />
+  <xacro:property name="arm_mount_rpy" value="0 0 3.141593" />
   <!-- Base: Ranger Mini 3.0 -->
   <xacro:include filename="$(find ranger_mini_v3_description)/urdf/ranger_mini_v3.xacro" />
