Commit message: Add UFACTORY F/T sensor variant and G2 gripper; remove superseded tool_head_link
model1300="true" on the xarm_device call swaps link6's mesh to
xarm_description's end_tool_1300 model (the F/T-sensor-equipped tool
flange) -- confirmed as the correct hardware variant by
RM_Version_1.2_production.step's own arm node name, "xArm6(XI1300)_...".

add_gripper/gripper_version="G2" adds the real UFACTORY G2 gripper at
link_eef: full kinematic tree (base_link, knuckles, fingers, mimic
joints), its own ros2_control resource, and a
gripper_position_controller (config/ros2_controllers.yaml + launch
spawner) so it's commandable in Gazebo immediately, matching how the
arm itself is wired.

Removes tool_head_link (and meshes/tool_head.stl): it attached at the
same link_eef frame the real gripper now occupies, and was only ever a
provisional placeholder guess for the ambiguous STEP "Tool head" part.

Verified end-to-end: xacro/check_urdf clean, and a full Gazebo launch
shows all three controllers (joint_state_broadcaster,
arm_velocity_controller, gripper_position_controller) loading,
configuring, and activating without error.

Co-Authored-By: Claude Sonnet 5 <noreply@anthropic.com>

File: ranger_xarm6_description/robots/ranger_xarm6.urdf.xacro (robot description, xacro)
@@ -85,5 +85,16 @@
   <xacro:include filename="$(find ranger_mini_v3_description)/urdf/ranger_mini_v3.xacro" />
   <xacro:ranger_mini_v3 prefix="$(arg prefix)" />
-  <!-- Arm: xArm6, mounted on the base via the placeholder FT above -->
+  <!-- Arm: xArm6, mounted on the base via the placeholder FT above.
+       model1300="true": this unit is the F/T-sensor-equipped "XI1300"
+       variant (confirmed by RM_Version_1.2_production.step's own arm
+       node name, "xArm6(XI1300)_02022023"), swaps link6's mesh from
+       the plain xarm_description default to end_tool/visual/collision
+       end_tool_1300.stl, xarm_description's actual model of the
+       F/T-sensor-equipped tool flange (see xarm6.urdf.xacro's
+       model_num >= 1300 branch). add_gripper/gripper_version="G2":
+       adds the real, properly-modeled UFACTORY G2 gripper at link_eef
+       (own links/joints/meshes + mimic-jointed fingers + its own
+       ros2_control "XArmGripperSystem" resource, driven via
+       gripper_position_controller below). -->
   <xacro:include filename="$(find xarm_description)/urdf/xarm_device_macro.xacro" />
   <xacro:xarm_device
@@ -100,4 +111,7 @@
     robot_ip="$(arg robot_ip)"
     load_gazebo_plugin="false"
+    model1300="true"
+    add_gripper="true"
+    gripper_version="G2"
   />
   <!-- Arm-to-base mounting plate (visual/collision only, no new joint):
@@ -207,47 +221,9 @@
     <origin xyz="${extras_xyz}" rpy="${extras_rpy}" />
   </joint>
-  <!-- Tool head / end-effector adapter (visual/collision only, static):
-       RM_Version_1.2_production.step's "Tool head" node, a small
-       (~86x54x79mm) part on the wrist, absent from Gazebo until now.
-       Mounted at link_eef (== link6 exactly here: dof=6,
-       add_realsense_d435i=false in the xarm_device call above, so
-       xarm_device_macro.xacro's joint_eef has a zero offset), the
-       canonical tool-mount frame xarm_description itself defines.
-       xyz/rpy below are a placeholder identity offset, NOT measured:
-       unlike arm_mount_xyz/rpy, this one couldn't be derived from the
-       STEP file at all, because the individual per-joint STEP nodes
-       (J1..J6) turned out to use arbitrary CAD-native part origins that
-       don't correspond to the URDF's joint/flange frames (checked: J1's
-       node origin isn't at the arm's own mounting frame either), and this
-       STEP's arm isn't necessarily posed at the URDF's zero configuration,
-       so there's no clean way to solve for the true link6->tool_head
-       offset from geometry alone. Needs the same visual-tuning-in-Gazebo
-       treatment arm_mount_xyz/rpy got. -->
-  <xacro:property name="tool_head_xyz" value="0 0 0" />
-  <xacro:property name="tool_head_rpy" value="0 0 0" />
-  <link name="$(arg prefix)tool_head_link">
-    <visual>
-      <geometry>
-        <mesh filename="package://ranger_xarm6_description/meshes/tool_head.stl" />
-      </geometry>
-      <material name="tool_head_grey">
-        <color rgba="0.3 0.3 0.3 1" />
-      </material>
-    </visual>
-    <collision>
-      <geometry>
-        <mesh filename="package://ranger_xarm6_description/meshes/tool_head.stl" />
-      </geometry>
-    </collision>
-    <inertial>
-      <mass value="0.1" />
-      <inertia ixx="0.0001" ixy="0" ixz="0" iyy="0.0001" iyz="0" izz="0.0001" />
-    </inertial>
-  </link>
-  <joint name="$(arg prefix)tool_head_joint" type="fixed">
-    <parent link="$(arg prefix)link_eef" />
-    <child link="$(arg prefix)tool_head_link" />
-    <origin xyz="${tool_head_xyz}" rpy="${tool_head_rpy}" />
-  </joint>
+  <!-- tool_head_link (the provisional STEP "Tool head" mesh, a
+       placeholder identity-offset guess) has been removed: the real G2
+       gripper now attaches at link_eef instead (via add_gripper/
+       gripper_version="G2" above), and the two would have overlapped at
+       the same frame. meshes/tool_head.stl is no longer referenced. -->
   <xacro:property name="_is_gz_sim" value="${'$(arg ros2_control_plugin)' == 'gz_ros2_control/GazeboSimSystem'}" />
   <xacro:if value="${_is_gz_sim}">
@@ -301,12 +277,13 @@
     </ros2_control>
   </xacro:if>
-  <!-- F/T SENSOR (Gazebo simulation only). Assumed present for this
-       integration, per instruction: treat sim force/contact behaviour as
-       real. On actual hardware this must instead come from xArm6's optional
-       F/T sensor accessory (see ranger_xarm6.launch.py's sim:=false path,
-       which remaps 'uf_ftsensor_ext_states'); whether this physical unit
-       has that accessory installed is unconfirmed (not itemised in the ARTC
-       handover note), so don't assume the sim behaviour carries over to
-       hardware without checking. Mirrors the same gz-sim force_torque
+  <!-- F/T SENSOR (Gazebo simulation only): simulated physics force/torque
+       measurement at joint6. This is the sim-side sensor plugin, separate
+       from model1300="true" above (which swaps in the F/T-sensor-equipped
+       tool-flange MESH); the physical accessory's presence, previously
+       flagged here as unconfirmed, is now confirmed by
+       RM_Version_1.2_production.step's arm node itself being named
+       "xArm6(XI1300)_02022023". On actual hardware this comes from that
+       accessory via ranger_xarm6.launch.py's sim:=false path (remaps
+       'uf_ftsensor_ext_states'). Mirrors the same gz-sim force_torque
        sensor + flat 'force_torque' topic convention robotnik_description
        uses at UR5e's wrist_3 for Theron/Kairos (see rbtheron_plus.urdf.xacro),

Commit message: Add two frame-mounted RealSense D435i cameras (fixed_cam1/fixed_cam2)
Per RM_Version_1.2_production.step's "Camera_module_for_design" cluster:
"Realsense_Camera_module v2" and "Realsense_Camera_module
v1(Mirror)(Mirror)" sit at the exact same point (0.0mm position
difference) differing only by a 180deg rotation about one axis, i.e.
these are two real cameras mounted back-to-back at the same point
facing opposite directions, not unresolved design variants of one
camera like the rest of that cluster (already folded into extras_link)
turned out to be. Final intended hardware is 3 cameras total: these 2
D435i plus 1 Orbbec Gemini 2 on the wrist (replacing the arm's current
D435i eventually, software-side only for now).

Position/rotation derived the same way as extras_link/mount_plate_link:
STEP-measured offset from the xArm-Mounting plate's own native origin,
composed with the current mount_plate_xyz/rpy.

Built from xarm_description's own d435i_urdf macro (same one the wrist
camera uses) so these are fully functional Gazebo camera sensors, not
decoration -- each needs its own common_material call and a distinct
fixed_camN_ prefix to avoid colliding with the arm's own link_eef/
camera_link names.

Found and fixed the same "Sensors system loaded twice" crash class as
the earlier world-file fix, but from a different source this time:
realsense_gz (realsense.gazebo.xacro) bundles the per-camera sensor
tags together with the gz::sim::systems::Sensors plugin registration in
one macro, so calling it once per camera (as a naive copy of the wrist
camera's approach would) re-registers that system 2 more times on top
of the wrist camera's own registration, segfaulting Ogre2 the same way.
Added a local fixed_cam_sensor_tags macro with just the sensor
declarations (copied from realsense_gz), no plugin block, since one
registration already covers the whole simulation.

Verified: xacro/check_urdf clean, full Gazebo launch runs without
crashing across two separate runs, all three controllers activate, and
all three cameras' full topic sets (color/depth/infra1/infra2 +
camera_info + points, 30 topics total) are confirmed live on
gz-transport.

Co-Authored-By: Claude Sonnet 5 <noreply@anthropic.com>

File: ranger_xarm6_description/robots/ranger_xarm6.urdf.xacro (robot description, xacro)
@@ -278,4 +278,184 @@
     </gazebo>
   </xacro:if>
+  <!-- Two frame-mounted RealSense D435i cameras, per
+       RM_Version_1.2_production.step's "Camera_module_for_design"
+       cluster: "Realsense_Camera_module v2" and
+       "Realsense_Camera_module v1(Mirror)(Mirror)" sit at the EXACT same
+       point (checked: 0.0mm position difference) and differ only by a
+       180deg rotation about one axis, i.e. not two unresolved design
+       variants of one camera like the rest of that cluster (folded into
+       extras_link) turned out to be, but two real cameras mounted
+       back-to-back at the same point, facing opposite directions. Final
+       intended hardware, per instruction: 2x D435i here (this block) +
+       1x Orbbec Gemini 2 on the wrist (replacing the arm's own camera
+       eventually, software-side only for now, keeping the D435i mesh
+       there via add_realsense_d435i above until Gemini's own ROS
+       packages are wired up).
+       Position/rotation derived the same way as extras_link/
+       mount_plate_link: STEP-measured offset from the xArm-Mounting
+       plate's own native origin, composed with the current (user-tuned)
+       mount_plate_xyz/rpy.
+       Built from xarm_description's own d435i_urdf/realsense_gz macros
+       (same ones the wrist camera above uses) rather than a plain
+       mesh, so these are fully functional Gazebo camera sensors, not
+       just decoration; needs its own explicit includes here since
+       those macros were only pulled in earlier INSIDE xarm_device's own
+       macro body (out of scope for us, same issue common.link.xacro /
+       xarm_gripper_macro.xacro had). Each needs a distinct prefix to
+       avoid colliding with the arm's own link_eef/camera_link names;
+       d435i_urdf hardcodes its camera body link as "${prefix}link_eef"
+       (an odd name to inherit for a base-mounted camera that isn't an
+       end-effector, but that's the vendored macro's own naming, kept
+       for consistency rather than forking it). -->
+  <xacro:include filename="$(find xarm_description)/urdf/camera/realsense_d435i.urdf.xacro" />
+  <xacro:include filename="$(find xarm_description)/urdf/common/common.material.xacro" />
+  <xacro:property name="fixed_cam_xyz" value="0.142000 0 0.063120" />
+  <xacro:property name="fixed_cam1_rpy" value="1.570796 0 -1.570796" />
+  <xacro:property name="fixed_cam2_rpy" value="1.570796 0 1.570796" />
+  <!-- common_material defines "${prefix}Silver" etc.; the arm's own call
+       (inside xarm_device above) only covers "$(arg prefix)Silver", not
+       these cameras' own fixed_camN_ prefixes, so d435i_urdf's visual
+       mesh material reference would otherwise be left undefined. -->
+  <xacro:common_material prefix="$(arg prefix)fixed_cam1_" />
+  <xacro:common_material prefix="$(arg prefix)fixed_cam2_" />
+  <xacro:d435i_urdf prefix="$(arg prefix)fixed_cam1_" add_d435i_links="true" />
+  <joint name="$(arg prefix)fixed_cam1_joint" type="fixed">
+    <parent link="$(arg prefix)base_link" />
+    <child link="$(arg prefix)fixed_cam1_link_eef" />
+    <origin xyz="${fixed_cam_xyz}" rpy="${fixed_cam1_rpy}" />
+  </joint>
+  <xacro:d435i_urdf prefix="$(arg prefix)fixed_cam2_" add_d435i_links="true" />
+  <joint name="$(arg prefix)fixed_cam2_joint" type="fixed">
+    <parent link="$(arg prefix)base_link" />
+    <child link="$(arg prefix)fixed_cam2_link_eef" />
+    <origin xyz="${fixed_cam_xyz}" rpy="${fixed_cam2_rpy}" />
+  </joint>
+  <!-- Sensor tags only (no Sensors-system <plugin> block): realsense_gz
+       (realsense.gazebo.xacro) bundles BOTH the per-camera sensor
+       declarations AND the world-wide gz::sim::systems::Sensors plugin
+       registration in one macro, so calling it here as-is per camera
+       would (and, tested, did) re-register that system a 2nd and 3rd
+       time on top of the wrist camera's own call inside xarm_device,
+       hitting the exact same "Another item already exists with name:
+       scene" Ogre2 crash tested_world.world's own duplicate copy caused
+       earlier (see that file's comment). One Sensors registration
+       (still xarm_device's, for the wrist camera) covers the whole
+       simulation; these two only need the sensor tags themselves. -->
+  <xacro:macro name="fixed_cam_sensor_tags" params="prefix">
+    <gazebo reference="${prefix}camera_depth_frame">
+      <sensor name="${prefix}cameradepth" type="rgbd_camera">
+        <camera name="${prefix}camera">
+          <horizontal_fov>1.57</horizontal_fov>
+          <image>
+            <width>1280</width>
+            <height>720</height>
+            <format>L8</format>
+          </image>
+          <clip>
+            <near>0.1</near>
+            <far>100</far>
+          </clip>
+          <depth_camera>
+            <clip>
+              <near>0.1</near>
+              <far>10</far>
+            </clip>
+          </depth_camera>
+          <noise>
+            <type>gaussian</type>
+            <mean>0.0</mean>
+            <stddev>0.100</stddev>
+          </noise>
+        </camera>
+        <always_on>1</always_on>
+        <update_rate>30</update_rate>
+        <visualize>0</visualize>
+        <topic>${prefix}camera/depth</topic>
+      </sensor>
+    </gazebo>
+    <gazebo reference="${prefix}camera_color_frame">
+      <sensor name="${prefix}cameracolor" type="camera">
+        <camera name="${prefix}camera">
+          <horizontal_fov>1.57</horizontal_fov>
+          <image>
+            <width>1280</width>
+            <height>720</height>
+            <format>RGB_INT8</format>
+          </image>
+          <clip>
+            <near>0.1</near>
+            <far>100</far>
+          </clip>
+          <noise>
+            <type>gaussian</type>
+            <mean>0.0</mean>
+            <stddev>0.007</stddev>
+          </noise>
+          <camera_info_topic>${prefix}camera/color/camera_info</camera_info_topic>
+        </camera>
+        <always_on>1</always_on>
+        <update_rate>30</update_rate>
+        <visualize>1</visualize>
+        <topic>${prefix}camera/color/image_raw</topic>
+        <enable_metrics>true</enable_metrics>
+      </sensor>
+    </gazebo>
+    <gazebo reference="${prefix}camera_left_ir_frame">
+      <sensor name="${prefix}cameraired1" type="camera">
+        <camera name="${prefix}camera">
+          <horizontal_fov>1.57</horizontal_fov>
+          <image>
+            <width>1280</width>
+            <height>720</height>
+            <format>L_INT8</format>
+          </image>
+          <clip>
+            <near>0.1</near>
+            <far>100</far>
+          </clip>
+          <noise>
+            <type>gaussian</type>
+            <mean>0.0</mean>
+            <stddev>0.05</stddev>
+          </noise>
+          <camera_info_topic>${prefix}camera/infra1/camera_info</camera_info_topic>
+        </camera>
+        <always_on>1</always_on>
+        <update_rate>30</update_rate>
+        <visualize>0</visualize>
+        <topic>${prefix}camera/infra1/image_raw</topic>
+      </sensor>
+    </gazebo>
+    <gazebo reference="${prefix}camera_right_ir_frame">
+      <sensor name="${prefix}cameraired2" type="camera">
+        <camera name="${prefix}camera">
+          <horizontal_fov>1.57</horizontal_fov>
+          <image>
+            <width>1280</width>
+            <height>720</height>
+            <format>L_INT8</format>
+          </image>
+          <clip>
+            <near>0.1</near>
+            <far>100</far>
+          </clip>
+          <noise>
+            <type>gaussian</type>
+            <mean>0.0</mean>
+            <stddev>0.05</stddev>
+          </noise>
+          <camera_info_topic>${prefix}camera/infra2/camera_info</camera_info_topic>
+        </camera>
+        <always_on>1</always_on>
+        <update_rate>30</update_rate>
+        <visualize>0</visualize>
+        <topic>${prefix}camera/infra2/image_raw</topic>
+      </sensor>
+    </gazebo>
+  </xacro:macro>
+  <xacro:if value="${_is_gz_sim}">
+    <xacro:fixed_cam_sensor_tags prefix="$(arg prefix)fixed_cam1_" />
+    <xacro:fixed_cam_sensor_tags prefix="$(arg prefix)fixed_cam2_" />
+  </xacro:if>
   <!-- State-only ros2_control interface for the base's 4 steering + 4 wheel
        joints (see ranger_mini_v3.xacro's own header comment: they're left
