Commit message: Swap fixed cameras to bare D435i mesh; fix two resulting bugs
Per instruction: the two frame-mounted cameras' mesh
(d435_with_cam_stand.stl, via xarm_description's d435i_urdf) carries
xarm's own arm-mount stand baked in, correct for the wrist camera but
wrong here where these two have their own separate STEP-modeled
mounting bracket. Switched to ros-humble-realsense2-description's
sensor_d435i macro instead, which uses the bare d435.dae mesh (no
mount) and is the same macro most ROS RealSense integrations use;
wrist camera is untouched (its stand mesh is correct there).

Two bugs surfaced by the switch, both fixed:

1. gz-sim doesn't resolve 'package://' mesh URIs against
   AMENT_PREFIX_PATH the way robot_state_publisher/RViz do -- needs
   GZ_SIM_RESOURCE_PATH explicitly, which is empty by default. This
   repo's own meshes were never affected because xarm_device_macro.xacro
   deliberately uses absolute file://$(find ...) paths instead of
   package:// specifically for the gz-sim case, sidestepping the
   problem entirely -- but realsense2_description's own sensor_d435i
   doesn't do that, so its mesh silently failed to load in Gazebo
   (SceneManager.cc error in the log, no crash). Fixed generally in
   ranger_xarm6.launch.py: GZ_SIM_RESOURCE_PATH is now derived from
   AMENT_PREFIX_PATH at launch time, covering every ROS package's share
   dir at once, not just this one.

2. realsense2_description's sensor_d435i names its IR frames
   camera_infra1_frame/camera_infra2_frame; the Gazebo sensor tags
   (fixed_cam_sensor_tags, copied from xarm_description's own
   realsense_gz macro for the earlier d435i_urdf-based version) still
   referenced xarm's naming, camera_left_ir_frame/camera_right_ir_frame.
   A <gazebo reference> pointing at a link that doesn't exist doesn't
   error, it just silently drops that sensor -- caught only by checking
   `gz topic -l` against the expected topic list, not from the launch
   log (which stayed clean). Fixed by updating the two reference names.

Verified: xacro/check_urdf clean, full Gazebo launch runs without
error or crash, and gz topic -l confirms the complete expected topic
set (30 topics: 3 cameras x color/depth/infra1/infra2 x
image+camera_info, plus depth extras) all present and live.

Co-Authored-By: Claude Sonnet 5 <noreply@anthropic.com>

File: ranger_xarm6_description/robots/ranger_xarm6.urdf.xacro (robot description, xacro)
@@ -296,39 +296,31 @@
        plate's own native origin, composed with the current (user-tuned)
        mount_plate_xyz/rpy.
-       Built from xarm_description's own d435i_urdf/realsense_gz macros
-       (same ones the wrist camera above uses) rather than a plain
-       mesh, so these are fully functional Gazebo camera sensors, not
-       just decoration; needs its own explicit includes here since
-       those macros were only pulled in earlier INSIDE xarm_device's own
-       macro body (out of scope for us, same issue common.link.xacro /
-       xarm_gripper_macro.xacro had). Each needs a distinct prefix to
-       avoid colliding with the arm's own link_eef/camera_link names;
-       d435i_urdf hardcodes its camera body link as "${prefix}link_eef"
-       (an odd name to inherit for a base-mounted camera that isn't an
-       end-effector, but that's the vendored macro's own naming, kept
-       for consistency rather than forking it). -->
-  <xacro:include filename="$(find xarm_description)/urdf/camera/realsense_d435i.urdf.xacro" />
-  <xacro:include filename="$(find xarm_description)/urdf/common/common.material.xacro" />
+       Built from the standard ros-humble-realsense2-description package's
+       own sensor_d435i macro (apt package, not xarm_description's
+       d435i_urdf like the wrist camera above uses): that vendored one
+       hardcodes xarm's own arm-mount stand into the visual mesh
+       (d435_with_cam_stand.stl), correct for the wrist where that stand
+       is the real hardware, wrong here where these two have their own
+       separate STEP-modeled mounting bracket. realsense2_description's
+       sensor_d435i uses the bare d435.dae mesh (no mount baked in) and
+       is the same macro most ROS RealSense integrations use. It has no
+       Gazebo sensor plugin wiring of its own though (purely mechanical
+       description), so the fixed_cam_sensor_tags macro below still
+       supplies that, same as before; frame naming lines up automatically
+       since sensor_d435i's own "name" param becomes the "${name}_"
+       prefix on all its frames (depth_frame, color_frame, etc.), and
+       fixed_cam_sensor_tags's "prefix" param is applied the same way. -->
+  <xacro:include filename="$(find realsense2_description)/urdf/_d435i.urdf.xacro" />
   <xacro:property name="fixed_cam_xyz" value="0.142000 0 0.063120" />
   <xacro:property name="fixed_cam1_rpy" value="1.570796 0 -1.570796" />
   <xacro:property name="fixed_cam2_rpy" value="1.570796 0 1.570796" />
-  <!-- common_material defines "${prefix}Silver" etc.; the arm's own call
-       (inside xarm_device above) only covers "$(arg prefix)Silver", not
-       these cameras' own fixed_camN_ prefixes, so d435i_urdf's visual
-       mesh material reference would otherwise be left undefined. -->
-  <xacro:common_material prefix="$(arg prefix)fixed_cam1_" />
-  <xacro:common_material prefix="$(arg prefix)fixed_cam2_" />
-  <xacro:d435i_urdf prefix="$(arg prefix)fixed_cam1_" add_d435i_links="true" />
-  <joint name="$(arg prefix)fixed_cam1_joint" type="fixed">
-    <parent link="$(arg prefix)base_link" />
-    <child link="$(arg prefix)fixed_cam1_link_eef" />
+  <xacro:sensor_d435i parent="$(arg prefix)base_link" name="$(arg prefix)fixed_cam1_camera"
+    use_nominal_extrinsics="true" use_mesh="true">
     <origin xyz="${fixed_cam_xyz}" rpy="${fixed_cam1_rpy}" />
-  </joint>
-  <xacro:d435i_urdf prefix="$(arg prefix)fixed_cam2_" add_d435i_links="true" />
-  <joint name="$(arg prefix)fixed_cam2_joint" type="fixed">
-    <parent link="$(arg prefix)base_link" />
-    <child link="$(arg prefix)fixed_cam2_link_eef" />
+  </xacro:sensor_d435i>
+  <xacro:sensor_d435i parent="$(arg prefix)base_link" name="$(arg prefix)fixed_cam2_camera"
+    use_nominal_extrinsics="true" use_mesh="true">
     <origin xyz="${fixed_cam_xyz}" rpy="${fixed_cam2_rpy}" />
-  </joint>
+  </xacro:sensor_d435i>
   <!-- Sensor tags only (no Sensors-system <plugin> block): realsense_gz
        (realsense.gazebo.xacro) bundles BOTH the per-camera sensor
@@ -341,5 +333,15 @@
        earlier (see that file's comment). One Sensors registration
        (still xarm_device's, for the wrist camera) covers the whole
-       simulation; these two only need the sensor tags themselves. -->
+       simulation; these two only need the sensor tags themselves.
+       Reference frame names below (camera_depth_frame, camera_infra1_frame,
+       etc.) match realsense2_description's sensor_d435i naming (infra1/
+       infra2), NOT xarm_description's own d435i_urdf naming (left_ir/
+       right_ir) that this macro's sensor tag content was originally
+       copied from, and mismatched once already (silently: gz-sim doesn't
+       error on a <gazebo reference> pointing at a link that doesn't
+       exist, it just drops that sensor, so fixed_cam1/2's infra1/infra2
+       topics were simply missing with nothing in the log to explain why;
+       caught by checking `gz topic -l` against the expected topic list
+       rather than trusting a clean launch log alone). -->
   <xacro:macro name="fixed_cam_sensor_tags" params="prefix">
     <gazebo reference="${prefix}camera_depth_frame">
@@ -401,5 +403,5 @@
       </sensor>
     </gazebo>
-    <gazebo reference="${prefix}camera_left_ir_frame">
+    <gazebo reference="${prefix}camera_infra1_frame">
       <sensor name="${prefix}cameraired1" type="camera">
         <camera name="${prefix}camera">
@@ -427,5 +429,5 @@
       </sensor>
     </gazebo>
-    <gazebo reference="${prefix}camera_right_ir_frame">
+    <gazebo reference="${prefix}camera_infra2_frame">
       <sensor name="${prefix}cameraired2" type="camera">
         <camera name="${prefix}camera">

Commit message: Mount the two fixed D435i cameras at camera_module_for_design's centre height, with a real position offset
Height (Z) raised from the individual Realsense_Camera_module STEP
node's own position (0.06312m) to Camera_module_for_design's own
bbox-center height (0.3885m in base_link frame), computed the same way
as extras_link's own bbox-center placement but scoped to just that
STEP node (excludes COMPOUND004, the separate root-level leftover
bucket folded into extras_link).

Also gives the two cameras a real Y-position offset (+-0.034949m)
instead of the coincident placement they had before: in STEP the two
Realsense_Camera_module variants actually sit at the exact same point
(differing only by a 180deg rotation), but per instruction they need
a genuine position offset between them. Reused the USB camera pair's
own real measured left/right spacing from that same STEP cluster
(USB_Camera_module v2 / v1(Mirror), a genuine mounted pair) rather
than picking an arbitrary number.

User-tuned fixed_cam1_rpy/fixed_cam2_rpy left untouched.

Verified: xacro/check_urdf clean, full Gazebo launch runs without
error, all three controllers activate.

Co-Authored-By: Claude Sonnet 5 <noreply@anthropic.com>

File: ranger_xarm6_description/robots/ranger_xarm6.urdf.xacro (robot description, xacro)
@@ -280,11 +280,11 @@
   <!-- Two frame-mounted RealSense D435i cameras, per
        RM_Version_1.2_production.step's "Camera_module_for_design"
-       cluster: "Realsense_Camera_module v2" and
-       "Realsense_Camera_module v1(Mirror)(Mirror)" sit at the EXACT same
-       point (checked: 0.0mm position difference) and differ only by a
-       180deg rotation about one axis, i.e. not two unresolved design
-       variants of one camera like the rest of that cluster (folded into
-       extras_link) turned out to be, but two real cameras mounted
-       back-to-back at the same point, facing opposite directions. Final
+       cluster. In STEP, "Realsense_Camera_module v2" and
+       "Realsense_Camera_module v1(Mirror)(Mirror)" actually sit at the
+       exact same point (checked: 0.0mm position difference), differing
+       only by a 180deg rotation about one axis; per instruction, given a
+       real position offset instead (matching the USB camera pair's own
+       genuine left/right spacing in that same cluster, see fixed_cam1_xyz/
+       fixed_cam2_xyz below), rather than mounting them coincident. Final
        intended hardware, per instruction: 2x D435i here (this block) +
        1x Orbbec Gemini 2 on the wrist (replacing the arm's own camera
@@ -312,14 +312,28 @@
        fixed_cam_sensor_tags's "prefix" param is applied the same way. -->
   <xacro:include filename="$(find realsense2_description)/urdf/_d435i.urdf.xacro" />
-  <xacro:property name="fixed_cam_xyz" value="0.142000 0 0.063120" />
-  <xacro:property name="fixed_cam1_rpy" value="1.570796 0 -1.570796" />
-  <xacro:property name="fixed_cam2_rpy" value="1.570796 0 1.570796" />
+  <!-- Height (Z) raised from the individual Realsense_Camera_module STEP
+       node's own position (0.06312m) to Camera_module_for_design's own
+       bbox-center height (0.3885m in base_link frame; X/Y of that center
+       are ~0.142/~0, matching what was already used, so only Z actually
+       changes), per instruction: mount at the height of the whole
+       cluster's centre, not the individual camera part's own STEP
+       position. Y offset (+-0.034949m) reuses the USB camera pair's own
+       real measured left/right spacing in this same STEP cluster
+       (USB_Camera_module v2 / v1(Mirror), a genuine mounted pair, unlike
+       the two Realsense variants which sit exactly coincident in STEP,
+       see the comment below) rather than an arbitrary number, per
+       instruction that the two cameras need a real position offset
+       between them, not just the orientation difference they had before. -->
+  <xacro:property name="fixed_cam1_xyz" value="0.142000 0.034949 0.388500" />
+  <xacro:property name="fixed_cam2_xyz" value="0.142000 -0.034949 0.388500" />
+  <xacro:property name="fixed_cam1_rpy" value="0 0 0" />
+  <xacro:property name="fixed_cam2_rpy" value="0 0 3.14159" />
   <xacro:sensor_d435i parent="$(arg prefix)base_link" name="$(arg prefix)fixed_cam1_camera"
     use_nominal_extrinsics="true" use_mesh="true">
-    <origin xyz="${fixed_cam_xyz}" rpy="${fixed_cam1_rpy}" />
+    <origin xyz="${fixed_cam1_xyz}" rpy="${fixed_cam1_rpy}" />
   </xacro:sensor_d435i>
   <xacro:sensor_d435i parent="$(arg prefix)base_link" name="$(arg prefix)fixed_cam2_camera"
     use_nominal_extrinsics="true" use_mesh="true">
-    <origin xyz="${fixed_cam_xyz}" rpy="${fixed_cam2_rpy}" />
+    <origin xyz="${fixed_cam2_xyz}" rpy="${fixed_cam2_rpy}" />
   </xacro:sensor_d435i>
   <!-- Sensor tags only (no Sensors-system <plugin> block): realsense_gz

Commit message: Tune fixed camera positions per visual check in Gazebo
fixed_cam1_xyz/fixed_cam2_xyz adjusted from the symmetric-Y-offset
starting point (matching the USB camera pair's spacing) to an
asymmetric X/Y placement, same provisional workflow as the other
STEP-derived transforms in this file.

Co-Authored-By: Claude Sonnet 5 <noreply@anthropic.com>

File: ranger_xarm6_description/robots/ranger_xarm6.urdf.xacro (robot description, xacro)
@@ -325,6 +325,6 @@
        instruction that the two cameras need a real position offset
        between them, not just the orientation difference they had before. -->
-  <xacro:property name="fixed_cam1_xyz" value="0.142000 0.034949 0.388500" />
-  <xacro:property name="fixed_cam2_xyz" value="0.142000 -0.034949 0.388500" />
+  <xacro:property name="fixed_cam1_xyz" value="0.250000 0.006 0.378500" />
+  <xacro:property name="fixed_cam2_xyz" value="0.032000 -0.006 0.378500" />
   <xacro:property name="fixed_cam1_rpy" value="0 0 0" />
   <xacro:property name="fixed_cam2_rpy" value="0 0 3.14159" />

Commit message: Wire realsense2_camera for the two fixed D435i cameras, sim and real
- Bridge fixed_cam1/fixed_cam2's gz-sim sensor topics to ROS2 (color/
  infra1/infra2/depth+points), and launch the real realsense2_camera
  driver per camera for sim:=false, both landing on matching
  /{robot_id}/fixed_cam{1,2}_camera/... topics.
- Fix the depth sensor's optical_frame_id: gz-sim's rgbd_camera
  publishes point-cloud XYZ in the physical (non-optical) frame
  convention, not the rotated optical one its own SDF element name
  implies; verified empirically against tested_world.world's geometry
  and a row/column sweep for mirror flips.
- Share one RViz instance (point-cloud/image displays) as the digital-
  twin viewer for both sim and real hardware; no live Gazebo alongside
  real hardware, following the standard ROS/Nav2 pattern.
- Add a sim-only depth-test cylinder 0.5m in front of fixed_cam1 for
  verifying point-cloud alignment against a known target.

Co-Authored-By: Claude Sonnet 5 <noreply@anthropic.com>

File: ranger_xarm6_description/robots/ranger_xarm6.urdf.xacro (robot description, xacro)
@@ -362,4 +362,36 @@
       <sensor name="${prefix}cameradepth" type="rgbd_camera">
         <camera name="${prefix}camera">
+          <!-- Without this, gz-sim falls back to an auto-generated scoped
+               entity path (e.g. 'robot_a/robot_a_base_link/robot_a_fixed_cam1_cameradepth')
+               as the frame_id on every message this sensor publishes (image,
+               depth image, points, camera_info), not a real TF frame, so
+               RViz's PointCloud2/Image displays silently render nothing (no
+               transform found), even fully enabled. See camera.sdf's own
+               optical_frame_id element ("used in the camera_info message
+               header", though it's actually applied to all this sensor's
+               messages, not just camera_info; confirmed by echoing
+               '.../depth/points's header.frame_id before/after this fix).
+               Deliberately pointed at camera_depth_frame (the PHYSICAL,
+               non-optical-rotated mount frame), NOT camera_depth_optical_frame
+               despite that being the ROS/realsense2_camera-driver convention
+               for a depth point cloud: verified empirically (dumped
+               .../depth/points, transformed through TF into robot_a_odom,
+               compared against tested_world.world's known wall/floor
+               geometry) that gz-sim's rgbd_camera sensor (Harmonic, gz-sensors
+               8.2.2) actually emits point-cloud XYZ in the SENSOR's own local/
+               physical axes (X-forward, Z-up, matching camera_depth_frame),
+               NOT the rotated X-right/Y-down/Z-forward optical convention its
+               own "optical_frame_id" element name implies. Labeling it
+               camera_depth_optical_frame (matching data already in the
+               physical convention) made RViz apply that frame's extra
+               rotation on top of already-correct data, throwing the cloud
+               off (points ending up below the floor, etc). If a future
+               gz-sensors version fixes this upstream (starts actually
+               rotating point data into the optical frame to match what
+               "optical_frame_id" implies), this will need to flip back to
+               camera_depth_optical_frame: re-run the same empirical check
+               (raw x/y/z stats vs. known nearby world geometry) rather than
+               assuming either way. -->
+          <optical_frame_id>${prefix}camera_depth_frame</optical_frame_id>
           <horizontal_fov>1.57</horizontal_fov>
           <image>
@@ -393,4 +425,6 @@
       <sensor name="${prefix}cameracolor" type="camera">
         <camera name="${prefix}camera">
+          <!-- See the depth sensor's own comment above: same fix, same reason. -->
+          <optical_frame_id>${prefix}camera_color_optical_frame</optical_frame_id>
           <horizontal_fov>1.57</horizontal_fov>
           <image>
@@ -420,4 +454,6 @@
       <sensor name="${prefix}cameraired1" type="camera">
         <camera name="${prefix}camera">
+          <!-- See the depth sensor's own comment above: same fix, same reason. -->
+          <optical_frame_id>${prefix}camera_infra1_optical_frame</optical_frame_id>
           <horizontal_fov>1.57</horizontal_fov>
           <image>
@@ -446,4 +482,6 @@
       <sensor name="${prefix}cameraired2" type="camera">
         <camera name="${prefix}camera">
+          <!-- See the depth sensor's own comment above: same fix, same reason. -->
+          <optical_frame_id>${prefix}camera_infra2_optical_frame</optical_frame_id>
           <horizontal_fov>1.57</horizontal_fov>
           <image>
@@ -473,4 +511,52 @@
     <xacro:fixed_cam_sensor_tags prefix="$(arg prefix)fixed_cam1_" />
     <xacro:fixed_cam_sensor_tags prefix="$(arg prefix)fixed_cam2_" />
+  </xacro:if>
+  <!-- Sim-only depth-test target: a tall, slim, world-upright cylinder,
+       0.5m straight out from fixed_cam1's own lens, for visually/
+       numerically verifying that camera's point cloud alignment (an
+       asymmetric-enough, unambiguous target: unlike tested_world.world's
+       flat, left-right-symmetric wall, which can't reveal certain bugs,
+       e.g. a mirror flip, since it looks the same either way).
+       Parented directly to fixed_cam1_camera_link (NOT base_link) so "0.5m
+       in front of the camera" stays literally true regardless of where
+       fixed_cam1_xyz/rpy above end up being tuned to. xyz="0.5 0 0" is
+       exactly the "camera forward" axis in that link's own physical
+       (non-optical) convention: the same X-forward convention this
+       package's point-cloud optical_frame_id fix (fixed_cam_sensor_tags'
+       depth sensor, above) is keyed to, so a correctly-calibrated point
+       cloud should show this cylinder's surface at very close to x=0.5m in
+       the raw (sensor-local) depth data.
+       rpy="0 0 0" (no counter-rotation) relies on fixed_cam1_xyz/rpy only
+       ever applying pure YAW (0 or pi so far, see fixed_cam1_rpy/
+       fixed_cam2_rpy above): yaw alone keeps a cylinder's own Z axis
+       aligned with world Z (upright) regardless of heading, so this only
+       needs revisiting if a fixed camera ever gets pitch/roll added.
+       Visual only (no <collision>): a depth/rgbd camera sensor renders
+       from the visual mesh, not physics collision, so collision geometry
+       would add self-collision computation for zero benefit here. Debug
+       aid only: gated on _is_gz_sim so it never appears on the real
+       robot's model. -->
+  <xacro:if value="${_is_gz_sim}">
+    <xacro:property name="cam1_test_target_radius" value="0.025" />
+    <xacro:property name="cam1_test_target_height" value="1.0" />
+    <link name="$(arg prefix)fixed_cam1_test_target_link">
+      <visual>
+        <geometry>
+          <cylinder radius="${cam1_test_target_radius}" length="${cam1_test_target_height}" />
+        </geometry>
+        <material name="test_target_orange">
+          <color rgba="1.0 0.5 0.0 1" />
+        </material>
+      </visual>
+      <inertial>
+        <mass value="0.05" />
+        <inertia ixx="0.0001" ixy="0" ixz="0" iyy="0.0001" iyz="0" izz="0.0001" />
+      </inertial>
+    </link>
+    <joint name="$(arg prefix)fixed_cam1_test_target_joint" type="fixed">
+      <parent link="$(arg prefix)fixed_cam1_camera_link" />
+      <child link="$(arg prefix)fixed_cam1_test_target_link" />
+      <origin xyz="0.5 0 0" rpy="0 0 0" />
+    </joint>
   </xacro:if>
   <!-- State-only ros2_control interface for the base's 4 steering + 4 wheel
