Commit message: Wire the wrist Orbbec Gemini 2, sim and real, mesh unchanged
Mesh stays the existing D435i+stand placeholder (xarm_device's
add_realsense_d435i, untouched) -- no combined Gemini2+xArm-mount mesh
exists to swap in (orbbec_description only ships a bare camera body, same
situation realsense2_description is in for the two fixed cameras). Software
side wired the same way as fixed_cam1/fixed_cam2, applied to the wrist's
existing D435i frame chain (camera_link/camera_depth_frame/camera_color_frame/
camera_left_ir_frame/camera_right_ir_frame, from xarm_device_macro, xarm_ros2
submodule, unchanged).

- ranger_xarm6.urdf.xacro: new wrist_camera_sensor_tags macro, same
  optical_frame_id fix as fixed_cam_sensor_tags' depth sensor (gz-sim's
  rgbd_camera point-cloud convention quirk), on distinct sensor
  names/topics ('{prefix}wrist_camera/...') so it doesn't collide with
  xarm's own realsense_gz-registered sensors on the same frames. Those
  keep running unused/unbridged alongside -- deliberately not editing
  xarm_ros2/xarm_description/urdf/camera/realsense.gazebo.xacro to fix
  them directly, since xarm_ros2 is a git submodule and add_d435i_links
  ties "create these frames" and "register xarm's own sensor tags" to one
  flag with no way to separate them. No new Sensors-system plugin
  registration needed -- xarm's own realsense_gz call already did that
  once.
- ranger_xarm6.launch.py: sim bridges wrist_camera's topics (reuses
  _fixed_camera_bridge_args with cam_id 'wrist'). Real hardware includes
  orbbec_camera's own gemini2.launch.py (ros-humble-orbbec-camera,
  installed), publish_tf:=false, cloud_frame_id matched to this URDF's
  camera_depth_frame. UNTESTED against physical hardware; color/infra1/
  infra2 frame_id parity with this URDF wasn't confirmed (no override
  found in gemini2.launch.py's own args for those, unlike cloud_frame_id).
- ranger_xarm6.rviz: depth heatmap (on) + color image (off) displays,
  same convention as the fixed cameras.

Verified live: all 10 topics bridge and stream real data (color image,
32FC1 depth, point cloud frame_id resolves via TF); fixed_cam1/fixed_cam2
confirmed unaffected and still streaming normally, per instruction not to
touch them.

Co-Authored-By: Claude Sonnet 5 <noreply@anthropic.com>

File: ranger_xarm6_description/robots/ranger_xarm6.urdf.xacro (robot description, xacro)
@@ -606,4 +606,165 @@
     <xacro:fixed_cam_sensor_tags prefix="$(arg prefix)fixed_cam2_" />
   </xacro:if>
+  <!-- Wrist camera (Orbbec Gemini 2, software-side only for now: mesh
+       stays the D435i+stand placeholder, see the header comment's own
+       "software-side only" note and this session's mesh-recommendation
+       discussion: no combined Gemini2+xArm-mount mesh exists, swapping it
+       would drop the mount geometry entirely). Same wiring treatment as
+       fixed_cam1/fixed_cam2 (correct optical_frame_id, own topics, bridged
+       + real driver), applied to the wrist's EXISTING D435i frame chain
+       (camera_link/camera_depth_frame/camera_color_frame/camera_left_ir_frame/
+       camera_right_ir_frame, from xarm_device's add_realsense_d435i="true"
+       above, itself unchanged): "lens distance similar, thickness differs"
+       per instruction, i.e. treat it as a D435i-shaped stand-in for now.
+       Deliberately NOT editing xarm_ros2/xarm_description/urdf/camera/
+       realsense.gazebo.xacro to add its own missing optical_frame_id (the
+       same bug fixed_cam_sensor_tags' own comment above documents) :
+       xarm_ros2 is a git submodule (this repo's own established practice
+       already avoids touching it, see xarm_device's add_gripper comment
+       above), and add_d435i_links (default true, unchanged) ties "create
+       these frames" and "register xarm's own broken sensor tags for them"
+       to the same flag with no way to get one without the other. Instead:
+       this macro adds a SEPARATE, correctly-configured sensor set on the
+       SAME existing frames, with distinct sensor names/topics (no
+       collision with xarm's own "${prefix}camera..." ones): xarm's own
+       copy keeps running unused/unbridged alongside (a real but accepted
+       small extra render cost, one wrist camera, in exchange for not
+       touching the submodule). No new Sensors-system plugin registration
+       needed: xarm's own realsense_gz call (still active, add_d435i_links
+       unchanged) already registered it once, same reason
+       fixed_cam_sensor_tags' own sensor tags don't re-register it either. -->
+  <xacro:macro name="wrist_camera_sensor_tags" params="prefix">
+    <gazebo reference="${prefix}camera_depth_frame">
+      <sensor name="${prefix}wristcameradepth" type="rgbd_camera">
+        <camera name="${prefix}wristcamera">
+          <!-- Physical, not optical, frame: same gz-sim rgbd_camera
+               point-cloud convention quirk as fixed_cam_sensor_tags' own
+               depth sensor above: see that comment for the full
+               empirical verification. Same gz-sensors version, same
+               sensor type, so the same fix applies here without needing
+               to re-derive it, though this specific sensor's point cloud
+               hasn't been separately re-verified against known world
+               geometry the way fixed_cam1's was. -->
+          <optical_frame_id>${prefix}camera_depth_frame</optical_frame_id>
+          <horizontal_fov>1.57</horizontal_fov>
+          <image>
+            <width>1280</width>
+            <height>720</height>
+            <format>L8</format>
+          </image>
+          <clip>
+            <near>0.1</near>
+            <far>100</far>
+          </clip>
+          <depth_camera>
+            <clip>
+              <near>0.1</near>
+              <far>10</far>
+            </clip>
+          </depth_camera>
+          <noise>
+            <type>gaussian</type>
+            <mean>0.0</mean>
+            <stddev>0.100</stddev>
+          </noise>
+        </camera>
+        <always_on>1</always_on>
+        <update_rate>30</update_rate>
+        <visualize>0</visualize>
+        <topic>${prefix}wrist_camera/depth</topic>
+      </sensor>
+    </gazebo>
+    <gazebo reference="${prefix}camera_color_frame">
+      <sensor name="${prefix}wristcameracolor" type="camera">
+        <camera name="${prefix}wristcamera">
+          <optical_frame_id>${prefix}camera_color_optical_frame</optical_frame_id>
+          <horizontal_fov>1.57</horizontal_fov>
+          <image>
+            <width>1280</width>
+            <height>720</height>
+            <format>RGB_INT8</format>
+          </image>
+          <clip>
+            <near>0.1</near>
+            <far>100</far>
+          </clip>
+          <noise>
+            <type>gaussian</type>
+            <mean>0.0</mean>
+            <stddev>0.007</stddev>
+          </noise>
+          <camera_info_topic>${prefix}wrist_camera/color/camera_info</camera_info_topic>
+        </camera>
+        <always_on>1</always_on>
+        <update_rate>30</update_rate>
+        <visualize>1</visualize>
+        <topic>${prefix}wrist_camera/color/image_raw</topic>
+        <enable_metrics>true</enable_metrics>
+      </sensor>
+    </gazebo>
+    <!-- Reference links are camera_left_ir_frame/camera_right_ir_frame
+         (xarm_description's own d435i_urdf naming), but topics/optical
+         frames below still say "infra1"/"infra2": matching xarm's own
+         realsense_gz macro's identical left=infra1/right=infra2 convention
+         (and fixed_cam_sensor_tags'), so downstream consumers see the same
+         topic shape regardless of which camera it's from. -->
+    <gazebo reference="${prefix}camera_left_ir_frame">
+      <sensor name="${prefix}wristcameraired1" type="camera">
+        <camera name="${prefix}wristcamera">
+          <optical_frame_id>${prefix}camera_left_ir_optical_frame</optical_frame_id>
+          <horizontal_fov>1.57</horizontal_fov>
+          <image>
+            <width>1280</width>
+            <height>720</height>
+            <format>L_INT8</format>
+          </image>
+          <clip>
+            <near>0.1</near>
+            <far>100</far>
+          </clip>
+          <noise>
+            <type>gaussian</type>
+            <mean>0.0</mean>
+            <stddev>0.05</stddev>
+          </noise>
+          <camera_info_topic>${prefix}wrist_camera/infra1/camera_info</camera_info_topic>
+        </camera>
+        <always_on>1</always_on>
+        <update_rate>30</update_rate>
+        <visualize>0</visualize>
+        <topic>${prefix}wrist_camera/infra1/image_raw</topic>
+      </sensor>
+    </gazebo>
+    <gazebo reference="${prefix}camera_right_ir_frame">
+      <sensor name="${prefix}wristcameraired2" type="camera">
+        <camera name="${prefix}wristcamera">
+          <optical_frame_id>${prefix}camera_right_ir_optical_frame</optical_frame_id>
+          <horizontal_fov>1.57</horizontal_fov>
+          <image>
+            <width>1280</width>
+            <height>720</height>
+            <format>L_INT8</format>
+          </image>
+          <clip>
+            <near>0.1</near>
+            <far>100</far>
+          </clip>
+          <noise>
+            <type>gaussian</type>
+            <mean>0.0</mean>
+            <stddev>0.05</stddev>
+          </noise>
+          <camera_info_topic>${prefix}wrist_camera/infra2/camera_info</camera_info_topic>
+        </camera>
+        <always_on>1</always_on>
+        <update_rate>30</update_rate>
+        <visualize>0</visualize>
+        <topic>${prefix}wrist_camera/infra2/image_raw</topic>
+      </sensor>
+    </gazebo>
+  </xacro:macro>
+  <xacro:if value="${_is_gz_sim}">
+    <xacro:wrist_camera_sensor_tags prefix="$(arg prefix)" />
+  </xacro:if>
   <!-- Plain single-image gz sensor for one usb_camera_macro instance
        (left_camera/right_camera): same structure as fixed_cam_sensor_tags'

Commit message: Use real Orbbec Gemini 2 extrinsics for the wrist camera, mesh unchanged
Per instruction: mesh stays the D435i+stand placeholder (camera_link,
unchanged, still parented to link_eef via xarm_device's own
camera_link_joint), but the depth/color/left_ir/right_ir spacing these
frames encode now reflects the real Gemini 2, not xarm_description's
borrowed D435i numbers.

New orbbec_gemini2_extrinsics macro adds gemini_depth_frame/
gemini_color_frame/gemini_left_ir_frame/gemini_right_ir_frame (+ their
optical children) parented directly to camera_link, with joint origins
pulled verbatim from ros-humble-orbbec-description's gemini_2.urdf.xacro
(installed on this machine, real measured values, not placeholders):
depth/left_ir coincident at (0,0,0) (Gemini 2 also derives depth from one
IR sensor, same as D435i), right_ir at (0,-0.05,0), color at
(0.00191,-0.014,0.000005). Composed straight onto camera_link rather than
copying that file's own camera_depth_frame-as-parent chain verbatim,
since that frame is itself an identity transform from camera_link either
way.

New, distinctly-named frames rather than overriding xarm_description's
own camera_depth_frame/etc in place: same "git submodule, don't edit it"
constraint already documented for wrist_camera_sensor_tags' duplicate
sensor registration applies here too (d435i_urdf ties frame creation to
the same flag as the mesh, no override hook). wrist_camera_sensor_tags
and the real orbbec_camera driver's cloud_frame_id now point at the new
frames.

Verified live: TF matches Orbbec's values exactly (color 0.002/-0.014/0,
right_ir 0/-0.05/0, depth 0/0/0), point cloud frame_id is
gemini_depth_frame, data streams, mesh confirmed still
d435_with_cam_stand.stl.

Co-Authored-By: Claude Sonnet 5 <noreply@anthropic.com>

File: ranger_xarm6_description/robots/ranger_xarm6.urdf.xacro (robot description, xacro)
@@ -634,6 +634,61 @@
        unchanged) already registered it once, same reason
        fixed_cam_sensor_tags' own sensor tags don't re-register it either. -->
+  <!-- Real Orbbec Gemini 2 extrinsics (depth/color/left_ir/right_ir
+       spacing), NOT xarm_description's borrowed D435i ones: per
+       instruction, mesh stays the D435i+stand placeholder (kept as
+       camera_link, unchanged, still parented to link_eef via
+       xarm_device's own camera_link_joint) but the actual sensor-to-
+       sensor geometry these frames encode should reflect the real
+       hardware. Pulled directly from ros-humble-orbbec-description's
+       gemini_2.urdf.xacro (installed on this machine), which ships real
+       measured joint origins, not placeholders; composed onto
+       camera_link directly rather than copying that file's own
+       parent chain verbatim: its camera_color_joint/camera_right_ir_joint
+       parent from camera_depth_frame, but that frame is itself
+       xyz="0 0 0" rpy="0 0 0" relative to camera_link (see its own
+       camera_depth_joint), i.e. an identity transform, so composing
+       through it or going straight to camera_link gives identical
+       numbers either way; straight to camera_link is simpler and avoids
+       needing a whole separate depth_frame-as-parent link just to prove
+       that to a future reader.
+       New, distinctly-named frames (gemini_*), NOT overriding
+       xarm_description's own camera_depth_frame/camera_color_frame/
+       camera_left_ir_frame/camera_right_ir_frame in place: those are
+       created by the same d435i_urdf macro that adds the mesh (tied to
+       the SAME add_realsense_d435i/add_d435i_links flags, no override
+       hook), and xarm_ros2 is a git submodule this repo's own established
+       practice already avoids editing (see wrist_camera_sensor_tags' own
+       comment below on the exact same constraint for its sensor tags).
+       xarm's own camera_*_frame links stay in the tree, unused now (no
+       sensor tags reference them any more), same "small accepted cost,
+       not worth a submodule edit" tradeoff already made for the
+       duplicate sensor registration. -->
+  <xacro:macro name="orbbec_gemini2_extrinsics" params="prefix">
+    <xacro:macro name="_gemini_frame" params="name xyz">
+      <joint name="${prefix}gemini_${name}_joint" type="fixed">
+        <origin xyz="${xyz}" rpy="0 0 0" />
+        <parent link="${prefix}camera_link" />
+        <child link="${prefix}gemini_${name}_frame" />
+      </joint>
+      <link name="${prefix}gemini_${name}_frame" />
+      <joint name="${prefix}gemini_${name}_optical_joint" type="fixed">
+        <origin xyz="0 0 0" rpy="${-pi/2} 0 ${-pi/2}" />
+        <parent link="${prefix}gemini_${name}_frame" />
+        <child link="${prefix}gemini_${name}_optical_frame" />
+      </joint>
+      <link name="${prefix}gemini_${name}_optical_frame" />
+    </xacro:macro>
+    <!-- depth and left_ir are coincident (0,0,0) in Orbbec's own file too,
+         same "depth derives from one IR sensor" convention D435i uses. -->
+    <xacro:_gemini_frame name="depth" xyz="0 0 0" />
+    <xacro:_gemini_frame name="left_ir" xyz="0 0 0" />
+    <xacro:_gemini_frame name="right_ir" xyz="0 -0.05000000074505806 0" />
+    <xacro:_gemini_frame name="color" xyz="0.0019099999917671084 -0.01400499977171421 4.999999873689376e-06" />
+  </xacro:macro>
+  <xacro:if value="${_is_gz_sim}">
+    <xacro:orbbec_gemini2_extrinsics prefix="$(arg prefix)" />
+  </xacro:if>
   <xacro:macro name="wrist_camera_sensor_tags" params="prefix">
-    <gazebo reference="${prefix}camera_depth_frame">
+    <gazebo reference="${prefix}gemini_depth_frame">
       <sensor name="${prefix}wristcameradepth" type="rgbd_camera">
         <camera name="${prefix}wristcamera">
@@ -646,5 +701,5 @@
                hasn't been separately re-verified against known world
                geometry the way fixed_cam1's was. -->
-          <optical_frame_id>${prefix}camera_depth_frame</optical_frame_id>
+          <optical_frame_id>${prefix}gemini_depth_frame</optical_frame_id>
           <horizontal_fov>1.57</horizontal_fov>
           <image>
@@ -675,8 +730,8 @@
       </sensor>
     </gazebo>
-    <gazebo reference="${prefix}camera_color_frame">
+    <gazebo reference="${prefix}gemini_color_frame">
       <sensor name="${prefix}wristcameracolor" type="camera">
         <camera name="${prefix}wristcamera">
-          <optical_frame_id>${prefix}camera_color_optical_frame</optical_frame_id>
+          <optical_frame_id>${prefix}gemini_color_optical_frame</optical_frame_id>
           <horizontal_fov>1.57</horizontal_fov>
           <image>
@@ -703,14 +758,16 @@
       </sensor>
     </gazebo>
-    <!-- Reference links are camera_left_ir_frame/camera_right_ir_frame
-         (xarm_description's own d435i_urdf naming), but topics/optical
-         frames below still say "infra1"/"infra2": matching xarm's own
-         realsense_gz macro's identical left=infra1/right=infra2 convention
-         (and fixed_cam_sensor_tags'), so downstream consumers see the same
+    <!-- Reference links are the new gemini_left_ir_frame/gemini_right_ir_frame
+         (this macro's own orbbec_gemini2_extrinsics, above; left/right
+         naming kept consistent with xarm_description's own d435i_urdf
+         convention it replaces), but topics/optical frames below still say
+         "infra1"/"infra2": matching xarm's own realsense_gz macro's
+         identical left=infra1/right=infra2 convention (and
+         fixed_cam_sensor_tags'), so downstream consumers see the same
          topic shape regardless of which camera it's from. -->
-    <gazebo reference="${prefix}camera_left_ir_frame">
+    <gazebo reference="${prefix}gemini_left_ir_frame">
       <sensor name="${prefix}wristcameraired1" type="camera">
         <camera name="${prefix}wristcamera">
-          <optical_frame_id>${prefix}camera_left_ir_optical_frame</optical_frame_id>
+          <optical_frame_id>${prefix}gemini_left_ir_optical_frame</optical_frame_id>
           <horizontal_fov>1.57</horizontal_fov>
           <image>
@@ -736,8 +793,8 @@
       </sensor>
     </gazebo>
-    <gazebo reference="${prefix}camera_right_ir_frame">
+    <gazebo reference="${prefix}gemini_right_ir_frame">
       <sensor name="${prefix}wristcameraired2" type="camera">
         <camera name="${prefix}wristcamera">
-          <optical_frame_id>${prefix}camera_right_ir_optical_frame</optical_frame_id>
+          <optical_frame_id>${prefix}gemini_right_ir_optical_frame</optical_frame_id>
           <horizontal_fov>1.57</horizontal_fov>
           <image>
