Commit message: Add Livox Mid-360 3D LIDAR: mesh, gz sensor, sim/real bridge, RViz
Mounted on extras_link, 30mm above the HiPNUC IMU's own joint position
(same X/Y, Z+0.030). Real mesh (not a placeholder box): copied from a
sibling workspace's robotnik_sensors package, which Robotnik ships in
production for the same Mid-360 unit; this repo can't depend on a
package from an unrelated workspace so it's vendored here as its own
copy. Mount/native-origin frame split and real mesh-alignment offsets
(90deg visual roll, +36.5mm sensor origin) also come from Robotnik's own
sensor_livox_mid_360 macro. The data frame is named "livox_frame"
(unprefixed-matching), not "livox_mid360_frame", to line up with Weston
Robot's own reference mount (wr_devkit_mapping) and livox_ros_driver2's/
LIO-SAM's own default frame_id/lidarFrame values.

Range (0.2-40.0m) and update_rate (10Hz) are Weston Robot's own real
operational values for this sensor (wr_devkit_mapping's params.yaml),
per their reference. Vertical FOV (-7 to 52deg) is the real Mid-360
datasheet spec. horizontal/vertical sample counts (1200/32) reuse
Robotnik's own tuned gz-sim gpu_lidar grid-approximation resolution:
gpu_lidar fundamentally can't reproduce Livox's real non-repetitive
scanning pattern, so there's no "real" number to derive instead.

gz-sim's gpu_lidar sensor has no native point-cloud output (only
rgbd_camera does), and ros_gz_bridge's own LaserScan converter was tried
first and found to silently truncate a multi-vertical-channel scan down
to its first row (verified live: 1200x32 sensor -> exactly 1200 ranges
bridged, not 38400). scripts/gz_lidar_to_pointcloud.py (new) subscribes
to the raw gz topic directly via gz-transport instead (same bindings
base_pose_publisher.py already uses), reading gz.msgs.LaserScan's own
vertical_count/vertical_angle_min/max/step fields straight from each
message, and republishes a real sensor_msgs/PointCloud2. Verified live:
10350 valid points/scan, frame_id resolves via TF, range/Z bounds sane
(0.29-31.3m, -0.71 to 1.37m), no NaNs.

Real hardware (sim:=false) also wired: livox_ros_driver2 is already
vendored/built in this exact workspace (unlike the HiPNUC IMU driver),
so unlike that IMU, this isn't left as a "decision pending" -- launches
livox_ros_driver2_node directly (not its own launch_ROS2/*.py files,
which hardcode the Livox-proprietary CustomMsg format at import time)
with xfer_format=0 for plain PointCloud2, matching sim's topic/frame_id.
Network config (lidar/host IPs) is the vendored default, software-side
wiring only until real hardware is available.

Adds an RViz PointCloud2 display (off by default, Color Transformer:
Intensity per livox_ros_driver2's own convention for this sensor).

Co-Authored-By: Claude Sonnet 5 <noreply@anthropic.com>

File: ranger_xarm6_description/robots/ranger_xarm6.urdf.xacro (robot description, xacro)
@@ -349,4 +349,67 @@
     <child link="$(arg prefix)hipnuc_imu_data_frame" />
     <origin xyz="0 0 0" rpy="0 0 -1.570796" />
+  </joint>
+  <!-- Livox Mid-360 3D LIDAR (360deg horizontal, non-repetitive scanning),
+       mounted on extras_link, "30mm above the joint position of the
+       IMU": same X/Y as hipnuc_imu_xyz, Z = hipnuc_imu_xyz's own
+       0.2205 + 0.030 = 0.2505.
+       Real mesh (not a placeholder box, unlike the IMU): copied from a
+       sibling workspace's robotnik_sensors package (meshes/3d_lidar/
+       livox_mid_360.stl), which Robotnik ships in production for the
+       same Mid-360 unit on their own robots: own copy here since this
+       repo can't depend on a package from an unrelated workspace.
+       Two frames, same mount/native-origin split as the IMU above:
+       livox_mid360_link: MOUNT frame (hosts the mesh). Rotated +90deg
+       yaw relative to extras_link (cancels extras_rpy's own -90deg), so
+       it ends up identity-aligned with base_link, same choice as
+       hipnuc_imu_link and matching Weston Robot's own reference mount
+       (github.com/westonrobot/wr_devkit_mapping's robot.urdf.xacro:
+       livox_joint, zero rotation relative to base_link). Mesh visual/
+       collision origin rpy="1.57 0 0" and scale 0.001 are real,
+       Robotnik-measured mesh-alignment facts (STL authored in mm, needs
+       a 90deg roll to sit upright), not guessed.
+       livox_frame: the SENSOR's own real point-cloud origin, child of
+       livox_mid360_link, offset +0.0365 in local Z: also a real
+       Robotnik-measured value (their own sensor_livox_mid_360 macro's
+       ${frame_prefix}joint). Named "livox_frame" (not "livox_mid360_
+       frame"), unprefixed-matching Weston Robot's own robot.urdf.xacro
+       AND livox_ros_driver2's own default 'frame_id' ROS param and
+       LIO-SAM's default 'lidarFrame' config value, for drop-in
+       compatibility with their mapping/nav stacks later if ever vendored
+       here (wr_devkit_mapping, wr_devkit_navigation). -->
+  <xacro:property name="livox_mid360_xyz" value="0 0.04 0.2505" />
+  <xacro:property name="livox_mid360_rpy" value="0 0 1.570796" />
+  <link name="$(arg prefix)livox_mid360_link">
+    <visual>
+      <origin xyz="0 0 0" rpy="${pi/2} 0 0" />
+      <geometry>
+        <mesh filename="package://ranger_xarm6_description/meshes/livox_mid_360.stl" scale="0.001 0.001 0.001" />
+      </geometry>
+      <material name="livox_mid360_grey">
+        <color rgba="0.75 0.75 0.75 1" />
+      </material>
+    </visual>
+    <collision>
+      <origin xyz="0 0 0" rpy="${pi/2} 0 0" />
+      <geometry>
+        <mesh filename="package://ranger_xarm6_description/meshes/livox_mid_360.stl" scale="0.001 0.001 0.001" />
+      </geometry>
+    </collision>
+    <inertial>
+      <origin xyz="0 0 0.029" rpy="0 0 0" />
+      <mass value="0.265" />
+      <inertia ixx="0.00013" ixy="0" ixz="0" iyy="0.00013" iyz="0" izz="0.00016" />
+    </inertial>
+  </link>
+  <joint name="$(arg prefix)livox_mid360_joint" type="fixed">
+    <parent link="$(arg prefix)extras_link" />
+    <child link="$(arg prefix)livox_mid360_link" />
+    <origin xyz="${livox_mid360_xyz}" rpy="${livox_mid360_rpy}" />
+  </joint>
+  <link name="$(arg prefix)livox_frame" />
+  <joint name="$(arg prefix)livox_frame_joint" type="fixed">
+    <parent link="$(arg prefix)livox_mid360_link" />
+    <child link="$(arg prefix)livox_frame" />
+    <origin xyz="0 0 0.0365" rpy="0 0 0" />
   </joint>
   <!-- tool_head_link (the provisional STEP "Tool head" mesh, a
@@ -1170,3 +1233,86 @@
     </gazebo>
   </xacro:if>
+  <!-- Livox Mid-360 (gz-sim only): attached to livox_frame (the real
+       sensor-origin child frame, not the mount link: see that frame's
+       own comment above). gz-sim's gpu_lidar sensor type has no native
+       point-cloud output (checked: libgz-sensors8-gpu-lidar.so has zero
+       references to "points" anywhere, unlike libgz-sensors8-rgbd_camera
+       .so, which does: rgbd_camera is a special combined sensor class
+       purpose-built to also emit PointCloudPacked, gpu_lidar never was).
+       It only ever publishes a flat gz.msgs.LaserScan on <topic>.
+       ros_gz_bridge's own sensor_msgs/LaserScan converter was tried
+       first and turned out to silently truncate a multi-vertical-channel
+       scan down to just its first (horizontal-only) row: verified live,
+       a 1200x32 sensor bridged to ROS came through with exactly 1200
+       ranges, not 38400 (no "vertical" string anywhere in
+       libros_gz_bridge_lib.so hinted at this beforehand, but didn't
+       prove it either way). gz_lidar_to_pointcloud.py (new,
+       ranger_xarm6.launch.py) subscribes to the raw gz topic directly
+       via gz-transport instead (bypassing ros_gz_bridge for this one
+       sensor entirely), reading gz.msgs.LaserScan's own proto fields
+       (vertical_count, vertical_angle_min/max/step) straight from each
+       message rather than duplicating horizontal_samples/vertical_
+       samples/angle values as separate, easy-to-drift-out-of-sync
+       launch arguments.
+       <gz_frame_id> works the same way it does for hipnuc_imu_sensor
+       above (a generic gz-sensors8 Sensor-base-class override, not
+       lidar-specific): confirmed via the same static check (Lidar's own
+       compiled library calls Sensor::FrameId(), same as Imu's), verified
+       live once built.
+       No new Sensors-system <plugin> registration needed: gpu_lidar is a
+       rendering sensor (like the cameras), and gz::sim::systems::Sensors
+       is already registered once via the wrist camera above.
+       Range 0.2-40.0m and update_rate 10Hz are Weston Robot's own real
+       operational values for this exact sensor (github.com/westonrobot/
+       wr_devkit_mapping's params.yaml: "lidarMinRange: 0.2 ... 0.2 for
+       livox", "lidarMaxRange: 40.0 ... 40.0 for livox", livox_ros_
+       driver2's own launch file's publish_freq=10.0 default), not the
+       datasheet's own more optimistic max-range spec. Vertical FOV
+       (-7 to 52deg) is the real Mid-360 datasheet spec (Weston Robot's
+       own materials don't give an angular FOV number to prefer instead).
+       horizontal_samples/vertical_samples (1200/32) are Robotnik's own
+       proven gz-sim gpu_lidar grid-approximation resolution: gpu_lidar
+       fundamentally cannot reproduce Livox's real non-repetitive
+       scanning pattern (a uniform rectangular sample grid is the only
+       shape gpu_lidar can render), so there's no "real" number to derive
+       instead; reusing an already-tuned value beats guessing a new one.
+       Noise stddev 0.03 is likewise Robotnik's own tuned value, no
+       better real number available for this simulation approximation. -->
+  <xacro:if value="${_is_gz_sim}">
+    <gazebo reference="$(arg prefix)livox_frame">
+      <sensor name="$(arg prefix)livox_mid360_sensor" type="gpu_lidar">
+        <always_on>1</always_on>
+        <update_rate>10</update_rate>
+        <visualize>false</visualize>
+        <topic>$(arg prefix)livox/lidar_raw</topic>
+        <gz_frame_id>$(arg prefix)livox_frame</gz_frame_id>
+        <lidar>
+          <scan>
+            <horizontal>
+              <samples>1200</samples>
+              <resolution>1</resolution>
+              <min_angle>${-pi}</min_angle>
+              <max_angle>${pi}</max_angle>
+            </horizontal>
+            <vertical>
+              <samples>32</samples>
+              <resolution>1</resolution>
+              <min_angle>${radians(-7)}</min_angle>
+              <max_angle>${radians(52)}</max_angle>
+            </vertical>
+          </scan>
+          <range>
+            <min>0.2</min>
+            <max>40.0</max>
+            <resolution>1</resolution>
+          </range>
+          <noise>
+            <type>gaussian</type>
+            <mean>0.0</mean>
+            <stddev>0.03</stddev>
+          </noise>
+        </lidar>
+      </sensor>
+    </gazebo>
+  </xacro:if>
 </robot>

Commit message: Update Livox Mid-360 mount pose, document the new hand-tuned values
livox_mid360_xyz: "0 0.04 0.2505" -> "0 0.04 0.2805" (another 0.030m up
from the nominal "30mm above the IMU joint" position).
livox_mid360_rpy: "0 0 1.570796" -> "0 0 -1.570796" -- livox_mid360_link
no longer cancels extras_rpy's own -90deg yaw, so it's now 180deg
rotated in yaw relative to base_link rather than identity-aligned (still
fine functionally: the Mid-360 scans the full 360deg horizontally
either way, only the raw scan's angle-to-robot-front mapping shifts).

Updated the placement/rotation derivation comments to describe the
actual current values instead of the stale nominal ones. Verified live:
extras_link->livox_mid360_link TF now resolves to [0, 0.04, 0.2805] with
-90deg yaw exactly as set, point cloud still publishes correct frame_id
and sane data (10146 points, range 0.29-32.8m, no NaNs).

Co-Authored-By: Claude Sonnet 5 <noreply@anthropic.com>

File: ranger_xarm6_description/robots/ranger_xarm6.urdf.xacro (robot description, xacro)
@@ -351,7 +351,11 @@
   </joint>
   <!-- Livox Mid-360 3D LIDAR (360deg horizontal, non-repetitive scanning),
-       mounted on extras_link, "30mm above the joint position of the
-       IMU": same X/Y as hipnuc_imu_xyz, Z = hipnuc_imu_xyz's own
-       0.2205 + 0.030 = 0.2505.
+       mounted on extras_link. Nominal placement was "30mm above the
+       joint position of the IMU": same X/Y as hipnuc_imu_xyz, Z =
+       hipnuc_imu_xyz's own 0.2205 + 0.030 = 0.2505; livox_mid360_xyz's
+       actual value, "0 0.04 0.2805", is hand-tuned another 0.030 higher
+       than that nominal (same X/Y), a mounting-position choice, not
+       re-derived here (same treatment as hipnuc_imu_xyz's own hand-tuned
+       value above).
        Real mesh (not a placeholder box, unlike the IMU): copied from a
        sibling workspace's robotnik_sensors package (meshes/3d_lidar/
@@ -360,11 +364,17 @@
        repo can't depend on a package from an unrelated workspace.
        Two frames, same mount/native-origin split as the IMU above:
-       livox_mid360_link: MOUNT frame (hosts the mesh). Rotated +90deg
-       yaw relative to extras_link (cancels extras_rpy's own -90deg), so
-       it ends up identity-aligned with base_link, same choice as
-       hipnuc_imu_link and matching Weston Robot's own reference mount
-       (github.com/westonrobot/wr_devkit_mapping's robot.urdf.xacro:
-       livox_joint, zero rotation relative to base_link). Mesh visual/
-       collision origin rpy="1.57 0 0" and scale 0.001 are real,
+       livox_mid360_link: MOUNT frame (hosts the mesh). livox_mid360_rpy
+       is hand-tuned to "0 0 -1.570796" (same -90deg yaw as extras_rpy,
+       not cancelling it): combined with extras_link's own -90deg yaw,
+       livox_mid360_link ends up rotated 180deg in yaw relative to
+       base_link, NOT identity-aligned the way hipnuc_imu_link and Weston
+       Robot's own reference mount (github.com/westonrobot/
+       wr_devkit_mapping's robot.urdf.xacro: livox_joint, zero rotation
+       relative to base_link) are: a deliberate mounting-orientation
+       choice (e.g. connector/cable routing direction), not re-derived
+       here. Since the Mid-360 scans the full 360deg horizontally, this
+       yaw choice doesn't affect scan coverage, only which horizontal
+       angle in the raw scan corresponds to the robot's own front. Mesh
+       visual/collision origin rpy="1.57 0 0" and scale 0.001 are real,
        Robotnik-measured mesh-alignment facts (STL authored in mm, needs
        a 90deg roll to sit upright), not guessed.
@@ -378,6 +388,6 @@
        compatibility with their mapping/nav stacks later if ever vendored
        here (wr_devkit_mapping, wr_devkit_navigation). -->
-  <xacro:property name="livox_mid360_xyz" value="0 0.04 0.2505" />
-  <xacro:property name="livox_mid360_rpy" value="0 0 1.570796" />
+  <xacro:property name="livox_mid360_xyz" value="0 0.04 0.2805" />
+  <xacro:property name="livox_mid360_rpy" value="0 0 -1.570796" />
   <link name="$(arg prefix)livox_mid360_link">
     <visual>
