Commit message: Replace full-detail mesh colliders with CoACD convex decompositions
extras, mount plate, Livox/IMU mount, HiPNUC IMU and Livox Mid-360 used
their visual meshes as colliders (~157k tris total, 122k for extras
alone). scripts/generate_colliders.py now decomposes each with CoACD
into convex hulls (108 hulls, ~18.7k tris), one <collision> per hull
via generated robots/_colliders.xacro macros, so MoveIt/Gazebo treat
them as convex pieces. All visual surfaces stay within 0.5mm of the
hulls.

Co-Authored-By: Claude Opus 5.5 <noreply@anthropic.com>

File: ranger_xarm6_description/robots/ranger_xarm6.urdf.xacro (robot description, xacro)
@@ -82,4 +82,9 @@
   <xacro:property name="mount_plate_xyz" value="-0.218500 0 0.02000" />
   <xacro:property name="mount_plate_rpy" value="0 0 -1.570796" />
+  <!-- CoACD convex-decomposition colliders (collider_<mesh> macros, one
+       <collision> per convex hull) for this package's own meshes, used in
+       place of their full-detail visual meshes. Regenerate with
+       scripts/generate_colliders.py. -->
+  <xacro:include filename="$(find ranger_xarm6_description)/robots/_colliders.xacro" />
   <!-- Base: Ranger Mini 3.0 -->
   <xacro:include filename="$(find ranger_mini_v3_description)/urdf/ranger_mini_v3.xacro" />
@@ -328,9 +333,5 @@
       </material>
     </visual>
-    <collision>
-      <geometry>
-        <mesh filename="package://ranger_xarm6_description/meshes/xarm_mount_plate.stl" />
-      </geometry>
-    </collision>
+    <xacro:collider_xarm_mount_plate />
     <inertial>
       <mass value="0.3" />
@@ -404,9 +405,5 @@
       </material>
     </visual>
-    <collision>
-      <geometry>
-        <mesh filename="package://ranger_xarm6_description/meshes/extras_compressed.stl" />
-      </geometry>
-    </collision>
+    <xacro:collider_extras_compressed />
     <inertial>
       <mass value="0.5" />
@@ -460,10 +457,5 @@
       </material>
     </visual>
-    <collision>
-      <origin xyz="${livox_imu_mount_mesh_xyz}" rpy="0 0 0" />
-      <geometry>
-        <mesh filename="package://ranger_xarm6_description/meshes/livox_imu_mount.stl" scale="0.001 0.001 0.001" />
-      </geometry>
-    </collision>
+    <xacro:collider_livox_imu_mount xyz="${livox_imu_mount_mesh_xyz}" scale="0.001 0.001 0.001" />
     <inertial>
       <origin xyz="0 0 0.02" rpy="0 0 0" />
@@ -516,10 +508,5 @@
       </material>
     </visual>
-    <collision>
-      <origin xyz="${hipnuc_imu_mesh_xyz}" rpy="0 0 -1.570796" />
-      <geometry>
-        <mesh filename="package://ranger_xarm6_description/meshes/hipnuc_imu.stl" scale="0.001 0.001 0.001" />
-      </geometry>
-    </collision>
+    <xacro:collider_hipnuc_imu xyz="${hipnuc_imu_mesh_xyz}" rpy="0 0 -1.570796" scale="0.001 0.001 0.001" />
     <inertial>
       <mass value="0.075" />
@@ -584,10 +571,5 @@
       </material>
     </visual>
-    <collision>
-      <origin xyz="0 0 0" rpy="${pi/2} 0 0" />
-      <geometry>
-        <mesh filename="package://ranger_xarm6_description/meshes/livox_mid_360.stl" scale="0.001 0.001 0.001" />
-      </geometry>
-    </collision>
+    <xacro:collider_livox_mid_360 rpy="${pi/2} 0 0" scale="0.001 0.001 0.001" />
     <inertial>
       <origin xyz="0 0 0.029" rpy="0 0 0" />

Commit message: Simulate the Mid-360's built-in IMU and the Ranger's wheel odometry
Both publish what the real drivers publish, so fusion can be built and
tested in sim against the same topics.

- Mid-360 IMU: livox_imu_frame at the ICM-40609's position in the point
  cloud frame (11.0, 23.29, -44.12 mm, manual), a 200 Hz gz IMU with
  datasheet white noise, and gz_livox_imu.py publishing 'livox/imu' in
  livox_ros_driver2's format: acceleration in g, frame_id the literal
  "livox_frame". The teleported base gives Gazebo's IMUs no motion to
  sense (a 0.3 rad/s spin read 0.006 rad/s), so the node adds the base's
  angular velocity and the acceleration at the IMU's position from
  ground truth.
- Wheel odometry: base_pose_publisher.py publishes 'odom' at 50 Hz like
  ranger_base (twist in base_link, zero covariances, no TF): the true
  motion with a 2% linear / -3% angular scale error and white noise,
  integrated so it drifts. The truth goes out on 'ground_truth/odom'.

Co-Authored-By: Claude Opus 5.5 <noreply@anthropic.com>

File: ranger_xarm6_description/robots/ranger_xarm6.urdf.xacro (robot description, xacro)
@@ -637,4 +637,15 @@
     <child link="$(arg prefix)livox_frame" />
     <origin xyz="0 0 0.0365" rpy="0 0 0" />
+  </joint>
+  <!-- Mid-360's built-in IMU (ICM-40609): the chip sits at (11.0, 23.29,
+       -44.12) mm in point-cloud (livox_frame) coordinates, axes the same
+       as the point cloud's (Livox Mid-360 User Manual). The real driver
+       stamps its messages "livox_frame" regardless (see
+       gz_livox_imu.py); this frame is the lidar-IMU extrinsic. -->
+  <link name="$(arg prefix)livox_imu_frame" />
+  <joint name="$(arg prefix)livox_imu_joint" type="fixed">
+    <parent link="$(arg prefix)livox_frame" />
+    <child link="$(arg prefix)livox_imu_frame" />
+    <origin xyz="0.011 0.02329 -0.04412" rpy="0 0 0" />
   </joint>
   <!-- tool_head_link (the provisional STEP "Tool head" mesh, a
@@ -1316,4 +1327,17 @@
         <state_interface name="linear_acceleration.z"/>
       </sensor>
+      <!-- Same, for the Mid-360's built-in IMU (livox_imu_sensor). -->
+      <sensor name="$(arg prefix)livox_imu_sensor">
+        <state_interface name="orientation.x"/>
+        <state_interface name="orientation.y"/>
+        <state_interface name="orientation.z"/>
+        <state_interface name="orientation.w"/>
+        <state_interface name="angular_velocity.x"/>
+        <state_interface name="angular_velocity.y"/>
+        <state_interface name="angular_velocity.z"/>
+        <state_interface name="linear_acceleration.x"/>
+        <state_interface name="linear_acceleration.y"/>
+        <state_interface name="linear_acceleration.z"/>
+      </sensor>
     </ros2_control>
   </xacro:if>
@@ -1550,3 +1574,43 @@
     </gazebo>
   </xacro:if>
+  <!-- Mid-360 built-in IMU (gz-sim only), on livox_imu_frame. 200 Hz like
+       the real one. White noise from the ICM-40609-D datasheet over the
+       100 Hz Nyquist band: gyro 0.0045 deg/s/rtHz -> 7.9e-4 rad/s,
+       accel 100 ug/rtHz -> 9.8e-3 m/s^2. The turn-on biases (bias_stddev)
+       are a moderate guess for a factory-calibrated unit, not datasheet
+       values (its uncalibrated board-level tolerances, +-1 deg/s and
+       +-40 mg, are far larger). Published raw on '<prefix>livox/imu_raw';
+       gz_livox_imu.py republishes it the way livox_ros_driver2 does. -->
+  <xacro:macro name="_livox_imu_axis_noise" params="axis stddev bias_stddev">
+    <xacro:element xacro:name="${axis}">
+      <noise type="gaussian">
+        <mean>0.0</mean>
+        <stddev>${stddev}</stddev>
+        <bias_mean>0.0</bias_mean>
+        <bias_stddev>${bias_stddev}</bias_stddev>
+      </noise>
+    </xacro:element>
+  </xacro:macro>
+  <xacro:if value="${_is_gz_sim}">
+    <gazebo reference="$(arg prefix)livox_imu_frame">
+      <sensor name="$(arg prefix)livox_imu_sensor" type="imu">
+        <always_on>1</always_on>
+        <update_rate>200</update_rate>
+        <topic>$(arg prefix)livox/imu_raw</topic>
+        <gz_frame_id>$(arg prefix)livox_imu_frame</gz_frame_id>
+        <imu>
+          <angular_velocity>
+            <xacro:_livox_imu_axis_noise axis="x" stddev="7.9e-4" bias_stddev="1e-3" />
+            <xacro:_livox_imu_axis_noise axis="y" stddev="7.9e-4" bias_stddev="1e-3" />
+            <xacro:_livox_imu_axis_noise axis="z" stddev="7.9e-4" bias_stddev="1e-3" />
+          </angular_velocity>
+          <linear_acceleration>
+            <xacro:_livox_imu_axis_noise axis="x" stddev="9.8e-3" bias_stddev="0.02" />
+            <xacro:_livox_imu_axis_noise axis="y" stddev="9.8e-3" bias_stddev="0.02" />
+            <xacro:_livox_imu_axis_noise axis="z" stddev="9.8e-3" bias_stddev="0.02" />
+          </linear_acceleration>
+        </imu>
+      </sensor>
+    </gazebo>
+  </xacro:if>
 </robot>

Commit message: Compute the sim Mid-360 IMU from ground truth, not a Gazebo sensor
The base is kinematic (teleported), so the Gazebo chassis's own physics
motion isn't the robot's: between teleports it creeps on its passive
wheels, and the teleport that snaps it back carries no velocity. The
Gazebo IMU sensed only the creep, a one-sided rotation (-0.012 rad/s
during a straight crab, truth 0) that turned the EKF's heading 2.6 deg
in 6 s.

sim_livox_imu.py (replacing gz_livox_imu.py) computes the IMU from
ground_truth/odom at 200 Hz sim time: angular velocity, gravity's
reaction plus the acceleration at the IMU's position, rotated into
livox_imu_frame, with the same datasheet white noise and seeded turn-on
biases. Output unchanged: 'livox/imu' in livox_ros_driver2's format.
The Gazebo IMU sensor and its ros2_control entry are gone;
livox_imu_frame stays.

Same sim test as the EKF commit (4 m square of crabs and 90 deg spins,
an arc, a sideways crab): EKF heading error stays within 0.18-0.25 deg
throughout (was drifting to 3.5 deg), position 3.6 cm; wheel odometry
alone 14.0 cm / 13.4 deg.

Co-Authored-By: Claude Opus 5.5 <noreply@anthropic.com>

File: ranger_xarm6_description/robots/ranger_xarm6.urdf.xacro (robot description, xacro)
@@ -641,6 +641,7 @@
        -44.12) mm in point-cloud (livox_frame) coordinates, axes the same
        as the point cloud's (Livox Mid-360 User Manual). The real driver
-       stamps its messages "livox_frame" regardless (see
-       gz_livox_imu.py); this frame is the lidar-IMU extrinsic. -->
+       stamps its messages "livox_frame" regardless; this frame is the
+       lidar-IMU extrinsic. Simulated by sim_livox_imu.py, not by a Gazebo
+       sensor (see there). -->
   <link name="$(arg prefix)livox_imu_frame" />
   <joint name="$(arg prefix)livox_imu_joint" type="fixed">
@@ -1327,17 +1328,4 @@
         <state_interface name="linear_acceleration.z"/>
       </sensor>
-      <!-- Same, for the Mid-360's built-in IMU (livox_imu_sensor). -->
-      <sensor name="$(arg prefix)livox_imu_sensor">
-        <state_interface name="orientation.x"/>
-        <state_interface name="orientation.y"/>
-        <state_interface name="orientation.z"/>
-        <state_interface name="orientation.w"/>
-        <state_interface name="angular_velocity.x"/>
-        <state_interface name="angular_velocity.y"/>
-        <state_interface name="angular_velocity.z"/>
-        <state_interface name="linear_acceleration.x"/>
-        <state_interface name="linear_acceleration.y"/>
-        <state_interface name="linear_acceleration.z"/>
-      </sensor>
     </ros2_control>
   </xacro:if>
@@ -1574,43 +1562,3 @@
     </gazebo>
   </xacro:if>
-  <!-- Mid-360 built-in IMU (gz-sim only), on livox_imu_frame. 200 Hz like
-       the real one. White noise from the ICM-40609-D datasheet over the
-       100 Hz Nyquist band: gyro 0.0045 deg/s/rtHz -> 7.9e-4 rad/s,
-       accel 100 ug/rtHz -> 9.8e-3 m/s^2. The turn-on biases (bias_stddev)
-       are a moderate guess for a factory-calibrated unit, not datasheet
-       values (its uncalibrated board-level tolerances, +-1 deg/s and
-       +-40 mg, are far larger). Published raw on '<prefix>livox/imu_raw';
-       gz_livox_imu.py republishes it the way livox_ros_driver2 does. -->
-  <xacro:macro name="_livox_imu_axis_noise" params="axis stddev bias_stddev">
-    <xacro:element xacro:name="${axis}">
-      <noise type="gaussian">
-        <mean>0.0</mean>
-        <stddev>${stddev}</stddev>
-        <bias_mean>0.0</bias_mean>
-        <bias_stddev>${bias_stddev}</bias_stddev>
-      </noise>
-    </xacro:element>
-  </xacro:macro>
-  <xacro:if value="${_is_gz_sim}">
-    <gazebo reference="$(arg prefix)livox_imu_frame">
-      <sensor name="$(arg prefix)livox_imu_sensor" type="imu">
-        <always_on>1</always_on>
-        <update_rate>200</update_rate>
-        <topic>$(arg prefix)livox/imu_raw</topic>
-        <gz_frame_id>$(arg prefix)livox_imu_frame</gz_frame_id>
-        <imu>
-          <angular_velocity>
-            <xacro:_livox_imu_axis_noise axis="x" stddev="7.9e-4" bias_stddev="1e-3" />
-            <xacro:_livox_imu_axis_noise axis="y" stddev="7.9e-4" bias_stddev="1e-3" />
-            <xacro:_livox_imu_axis_noise axis="z" stddev="7.9e-4" bias_stddev="1e-3" />
-          </angular_velocity>
-          <linear_acceleration>
-            <xacro:_livox_imu_axis_noise axis="x" stddev="9.8e-3" bias_stddev="0.02" />
-            <xacro:_livox_imu_axis_noise axis="y" stddev="9.8e-3" bias_stddev="0.02" />
-            <xacro:_livox_imu_axis_noise axis="z" stddev="9.8e-3" bias_stddev="0.02" />
-          </linear_acceleration>
-        </imu>
-      </sensor>
-    </gazebo>
-  </xacro:if>
 </robot>
