Commit message: Add sequential and whole-body MoveIt control for the Ranger + xArm6
The base only crabs (fixed heading) or spins in place, never both, to
match the Ranger's steering modes.

- moveit_config: MoveIt's URDF models the base as base_x/y/theta joints
  (plus a never-planned base_z) instead of a planar virtual joint, fed
  from odom -> base_link TF by base_joint_state_publisher.py. Groups
  base_translation, base_rotation and whole_body (x, y + arm); base
  joint limits; base_trajectory_controller in moveit_controllers.
- manipulation: control.launch.py (controller:=moveit_sequential |
  moveit_whole_body, declared choices) replaces manipulation.launch.py.
  MoveToGoal modes are DEFAULT=0, SEQUENTIAL=1, WHOLE_BODY=2.
  Coordinator plans every base move with OMPL; WHOLE_BODY spins first,
  then crabs and moves the arm in one plan, choosing the base position
  for pose goals when none is given. Applies a default 0.3 velocity
  scaling (move_group treated 0 as full speed), checks goal states for
  collisions up front, waits for the arm to settle before planning.
  base_trajectory_server.py tracks MoveIt trajectories in time and
  rejects any that both translate and rotate.
- description: world_collision_objects.py publishes the Gazebo world's
  static models to MoveIt's planning scene from the bringup.
  base_pose_publisher.py teleports only when driving or drifted, at the
  height Gazebo reports: teleporting a parked base to z every 33ms
  dropped it ~1cm each time and shook the arm (up to 7 rad/s).

Co-Authored-By: Claude Opus 5.5 <noreply@anthropic.com>

File: ranger_xarm6_moveit_config/srdf/ranger_xarm6.srdf.xacro (robot description, xacro)
@@ -6,11 +6,12 @@
   <xacro:arg name="prefix" default="" />
   <xacro:property name="prefix" value="$(arg prefix)" />
-  <!-- The mobile base as a planar joint (x, y, yaw) between odom and
-       base_link. MoveIt reads its value from TF (odom -> base_link, owned by
-       base_pose_publisher.py in sim, the Ranger driver on hardware), so the
-       planning scene always has the robot where it really is. Planned only
-       by the 'base' group; 'arm' plans with the base held still. -->
-  <virtual_joint name="${prefix}base_virtual_joint" type="planar"
-    parent_frame="${prefix}odom" child_link="${prefix}base_link" />
+  <!-- The mobile base is joints in MoveIt's URDF
+       (urdf/ranger_xarm6_moveit.urdf.xacro): base_x_joint, base_y_joint,
+       base_theta_joint (planned below) and base_z_joint (height, never
+       planned: passive), odom -> base_link. Their states come from TF
+       (odom -> base_link, via base_joint_state_publisher.py), so the
+       planning scene always has the robot where it really is. The groups
+       below never mix translation and rotation, the Ranger can't do both
+       in one steering mode (see that URDF). -->
   <group name="arm">
     <chain base_link="${prefix}link_base" tip_link="${prefix}link_tcp" />
@@ -26,6 +27,17 @@
     <joint name="${prefix}drive_joint" />
   </group>
-  <group name="base">
-    <joint name="${prefix}base_virtual_joint" />
+  <!-- Crab: translate at a fixed heading (Ranger parallel mode). -->
+  <group name="base_translation">
+    <joint name="${prefix}base_x_joint" />
+    <joint name="${prefix}base_y_joint" />
+  </group>
+  <!-- Spin in place (Ranger spinning mode). -->
+  <group name="base_rotation">
+    <joint name="${prefix}base_theta_joint" />
+  </group>
+  <!-- Base and arm together: crab + arm, heading locked. -->
+  <group name="whole_body">
+    <group name="base_translation" />
+    <group name="arm" />
   </group>
   <!-- home: xArm's own zero pose (gripper hangs down ~0.25m past the rear
@@ -66,4 +78,5 @@
        (follow drive_joint). Keep the wheel list in sync with
        scripts/generate_collision_matrix.py's PASSIVE_JOINTS. -->
+  <passive_joint name="${prefix}base_z_joint" />
   <passive_joint name="${prefix}fr_steering_joint" />
   <passive_joint name="${prefix}fr_wheel" />
