Commit message: Damp the Ranger's passive wheels and drive the gripper fingers in sim
- ranger_mini_v3: damping and friction on the 4 steering and 4 wheel
  joints. Nothing drives them (the base is teleported), so while
  parked the steering joints swung at ~1 rad/s and the wheels rolled.
  Sim only; the base's motion is unchanged.
- ranger_xarm6: in Gazebo, the five finger/knuckle joints join
  drive_joint's ros2_control block as gz_ros2_control mimic joints.
  xarm_gripper_macro's Gazebo Classic mimic plugin never loads in
  gz-sim, and gz-sim's own mimic constraint needs bullet-featherstone,
  so only the outer knuckle moved. The macro's parts are now called
  one by one; real hardware still gets no gripper block.

Co-Authored-By: Claude Opus 5.5 <noreply@anthropic.com>

File: ranger_mini_v3_description/urdf/ranger_mini_v3.xacro (robot description, xacro)
@@ -26,4 +26,16 @@
 <robot xmlns:xacro="http://ros.org/wiki/xacro">
   <xacro:macro name="ranger_mini_v3" params="prefix">
+    <!-- Joint damping [N*m*s/rad] and Coulomb friction [N*m] for the
+         passive steering/wheel joints, simulation only (the real driver
+         and MoveIt ignore <dynamics>). Nothing drives these joints: in sim
+         the base is teleported (base_pose_publisher.py), so without them
+         the steering joints swung freely (~1 rad/s) and the wheels rolled
+         while parked, and the arm's reaction forces rolled the chassis.
+         They don't change how the base moves when driving, that's the
+         teleport's. -->
+    <xacro:property name="steering_damping" value="5.0" />
+    <xacro:property name="steering_friction" value="2.0" />
+    <xacro:property name="wheel_damping" value="1.0" />
+    <xacro:property name="wheel_friction" value="1.0" />
     <link name="${prefix}base_link">
       <inertial>
@@ -106,4 +118,5 @@
         xyz="0 0 -1" />
       <limit effort="5" velocity="6.28"  lower="-2.1" upper="2.1" />
+      <dynamics damping="${steering_damping}" friction="${steering_friction}" />
     </joint>
     <link name="${prefix}fr_wheel_link">
@@ -136,4 +149,5 @@
       <child link="${prefix}fr_wheel_link"/>
       <axis xyz="0 1 0" rpy="0 0 0" />
+      <dynamics damping="${wheel_damping}" friction="${wheel_friction}" />
     </joint>
     <link name="${prefix}fl_steering_wheel_link">
@@ -187,4 +201,5 @@
         xyz="0 0 -1" />
       <limit effort="5" velocity="6.28"  lower="-2.1" upper="2.1" />
+      <dynamics damping="${steering_damping}" friction="${steering_friction}" />
     </joint>
     <link name="${prefix}fl_wheel_link">
@@ -217,4 +232,5 @@
       <child link="${prefix}fl_wheel_link"/>
       <axis xyz="0 1 0" rpy="0 0 0" />
+      <dynamics damping="${wheel_damping}" friction="${wheel_friction}" />
     </joint>
     <link name="${prefix}rl_steering_wheel_link">
@@ -268,4 +284,5 @@
         xyz="0 0 -1" />
       <limit effort="5" velocity="6.28"  lower="-2.1" upper="2.1" />
+      <dynamics damping="${steering_damping}" friction="${steering_friction}" />
     </joint>
     <link name="${prefix}rl_wheel_link">
@@ -298,4 +315,5 @@
       <child link="${prefix}rl_wheel_link"/>
       <axis xyz="0 1 0" rpy="0 0 0" />
+      <dynamics damping="${wheel_damping}" friction="${wheel_friction}" />
     </joint>
     <link name="${prefix}rr_steering_wheel_link">
@@ -326,4 +344,5 @@
       <axis xyz="0 0 -1" rpy="0 0 0" />
       <limit effort="5" velocity="6.28"  lower="-2.1" upper="2.1" />
+      <dynamics damping="${steering_damping}" friction="${steering_friction}" />
     </joint>
     <link name="${prefix}rr_wheel_link">
@@ -356,4 +375,5 @@
       <child link="${prefix}rr_wheel_link"/>
       <axis xyz="0 1 0" rpy="0 0 0" />
+      <dynamics damping="${wheel_damping}" friction="${wheel_friction}" />
     </joint>
   </xacro:macro>

File: ranger_xarm6_description/robots/ranger_xarm6.urdf.xacro (robot description, xacro)
@@ -307,15 +307,64 @@
        hard_interface left at its default (PositionJointInterface,
        matching effort_control=false/velocity_control=false,
-       xarm_device's own defaults, which the arm above also used). -->
+       xarm_device's own defaults, which the arm above also used).
+       xarm_gripper_macro's own parts are called one by one instead of the
+       macro itself, so that in Gazebo the five finger/knuckle joints can
+       join drive_joint's ros2_control block (below). The macro follows
+       drive_joint with libgazebo_mimic_joint_plugin.so, a Gazebo Classic
+       plugin gz-sim never loads, and gz-sim's own mimic constraint (from
+       the URDF <mimic> tags) needs bullet-featherstone, not DART, which
+       it logs as "the chosen physics engine does not support mimic
+       constraints": without either, only drive_joint's outer knuckle moved
+       and the fingers hung loose. -->
   <xacro:include filename="$(find xarm_description)/urdf/gripper/xarm_gripper_macro.xacro" />
-  <xacro:xarm_gripper_macro
+  <xacro:xarm_gripper_urdf
     prefix="$(arg prefix)"
     attach_to="$(arg prefix)camera_mount_link"
     attach_xyz="0 0 0.003"
     attach_rpy="0 0 0"
-    ros2_control_plugin="$(arg ros2_control_plugin)"
-    dof="6"
     gripper_version="G2"
   />
+  <xacro:xarm_gripper_transmission prefix="$(arg prefix)" />
+  <xacro:xarm_gripper_gazebo prefix="$(arg prefix)" />
+  <!-- Gazebo: gz_ros2_control's own mimic joints (a 'mimic' param on a
+       joint in the same <ros2_control> block as the joint it follows)
+       drive each finger/knuckle joint to drive_joint's position every
+       update, on any physics engine. They show up in joint_states as
+       '<joint>_mimic'; robot_state_publisher still places the fingers from
+       drive_joint via the URDF <mimic> tags. Real hardware
+       (UFRobotSystemHardware): no gripper block, same as
+       xarm_gripper_macro; any other plugin (fake hardware): its block. -->
+  <xacro:if value="${'$(arg ros2_control_plugin)' == 'gz_ros2_control/GazeboSimSystem'}">
+    <ros2_control name="$(arg prefix)XArmGripperSystem" type="system">
+      <hardware>
+        <plugin>gz_ros2_control/GazeboSimSystem</plugin>
+      </hardware>
+      <joint name="$(arg prefix)drive_joint">
+        <command_interface name="position" />
+        <command_interface name="velocity">
+          <param name="min">-3.14</param>
+          <param name="max">3.14</param>
+        </command_interface>
+        <state_interface name="position" />
+        <state_interface name="velocity" />
+      </joint>
+      <xacro:macro name="_gripper_mimic_joint" params="name">
+        <joint name="$(arg prefix)${name}">
+          <param name="mimic">$(arg prefix)drive_joint</param>
+          <param name="multiplier">1</param>
+          <state_interface name="position" />
+          <state_interface name="velocity" />
+        </joint>
+      </xacro:macro>
+      <xacro:_gripper_mimic_joint name="left_finger_joint" />
+      <xacro:_gripper_mimic_joint name="left_inner_knuckle_joint" />
+      <xacro:_gripper_mimic_joint name="right_outer_knuckle_joint" />
+      <xacro:_gripper_mimic_joint name="right_finger_joint" />
+      <xacro:_gripper_mimic_joint name="right_inner_knuckle_joint" />
+    </ros2_control>
+  </xacro:if>
+  <xacro:unless value="${'$(arg ros2_control_plugin)' in ('gz_ros2_control/GazeboSimSystem', 'uf_robot_hardware/UFRobotSystemHardware')}">
+    <xacro:xarm_gripper_ros2_control prefix="$(arg prefix)" ros2_control_plugin="$(arg ros2_control_plugin)" />
+  </xacro:unless>
   <!-- Arm-to-base mounting plate (visual/collision only, no new joint):
        the physical bracket the xArm6 bolts to on top of the Ranger, per

Commit message: Sim base driven by its wheels through gz_ros2_control
The sim base was teleported along cmd_vel (base_pose_publisher.py): no
slip, no inertia, through walls, and nothing it carried came along. Now
(base_drive:=physics, the default) gz_ros2_control drives the 4 steering
joints (position) and 4 wheels (velocity), and ranger_sim_base.py stands
in for the real driver:

- cmd_vel -> wheels with the real driver's motion modes
  (westonrobot_ranger_ros2 TwistCmdCallback): crab when linear.y != 0,
  spin in place under a 0.476 m turn radius (vx ignored), dual Ackermann
  otherwise; wheel positions from TF (rear-right isn't symmetric).
  Wheels change speed at most 1 m/s^2; a big re-steer (> 0.5 rad, a mode
  change) brakes to a stop on the old angles first, smaller ones steer
  while driving. Stopping the wheels at once locked them and the base
  skidded on; stopping for every small re-aim left MoveIt's docking
  corrections short of the dock.
- wheel odometry on 'odom' from the measured wheel states (least
  squares), in the real driver's format, plus the same scale error and
  noise as before;
- odom -> base_link TF and ground_truth/odom from Gazebo's
  OdometryPublisher (true motion).

ranger_mini_v3 macro param 'driven': steering effort 30 N.m and light
damping when driven (the passive values used up the 5 N.m at ~0.6 rad/s).
base_drive:=kinematic keeps the old teleported base.

Sim: DemoPickPlace SUCCESS (391 s); parked drift 0; RTF 0.82 vs 0.86.

Co-Authored-By: Claude Opus 5.5 <noreply@anthropic.com>
Claude-Session: https://claude.ai/code/session_01J4zo453gEdwitfs3w5jzWy

File: ranger_mini_v3_description/urdf/ranger_mini_v3.xacro (robot description, xacro)
@@ -25,17 +25,24 @@
 -->
 <robot xmlns:xacro="http://ros.org/wiki/xacro">
-  <xacro:macro name="ranger_mini_v3" params="prefix">
-    <!-- Joint damping [N*m*s/rad] and Coulomb friction [N*m] for the
-         passive steering/wheel joints, simulation only (the real driver
-         and MoveIt ignore <dynamics>). Nothing drives these joints: in sim
-         the base is teleported (base_pose_publisher.py), so without them
-         the steering joints swung freely (~1 rad/s) and the wheels rolled
-         while parked, and the arm's reaction forces rolled the chassis.
-         They don't change how the base moves when driving, that's the
-         teleport's. -->
-    <xacro:property name="steering_damping" value="5.0" />
-    <xacro:property name="steering_friction" value="2.0" />
-    <xacro:property name="wheel_damping" value="1.0" />
-    <xacro:property name="wheel_friction" value="1.0" />
+  <!-- driven: the steering joints and wheels are commanded in sim
+       (ranger_xarm6's sim_base_drive physics), else passive. -->
+  <xacro:macro name="ranger_mini_v3" params="prefix driven:=false">
+    <!-- Joint damping [N*m*s/rad], Coulomb friction [N*m] and the steering
+         joints' effort limit [N*m], simulation only (the real driver and
+         MoveIt ignore <dynamics> and effort).
+         Passive (the base teleported, base_pose_publisher.py): nothing
+         holds these joints, so without damping and friction the steering
+         joints swung freely (~1 rad/s) and the wheels rolled while parked,
+         and the arm's reaction forces rolled the chassis.
+         Driven (ranger_sim_base.py): the controllers hold them, and the
+         steering motors must overcome the tyres' scrub: with the passive
+         values, damping + friction used up the whole 5 N*m at ~0.6 rad/s
+         and a steering joint dragged by the others couldn't reach its
+         angle at all. -->
+    <xacro:property name="steering_damping" value="${0.5 if driven else 5.0}" />
+    <xacro:property name="steering_friction" value="${0.2 if driven else 2.0}" />
+    <xacro:property name="steering_effort" value="${30 if driven else 5}" />
+    <xacro:property name="wheel_damping" value="${0.05 if driven else 1.0}" />
+    <xacro:property name="wheel_friction" value="${0.05 if driven else 1.0}" />
     <link name="${prefix}base_link">
       <inertial>
@@ -117,5 +124,5 @@
       <axis
         xyz="0 0 -1" />
-      <limit effort="5" velocity="6.28"  lower="-2.1" upper="2.1" />
+      <limit effort="${steering_effort}" velocity="6.28"  lower="-2.1" upper="2.1" />
       <dynamics damping="${steering_damping}" friction="${steering_friction}" />
     </joint>
@@ -200,5 +207,5 @@
       <axis
         xyz="0 0 -1" />
-      <limit effort="5" velocity="6.28"  lower="-2.1" upper="2.1" />
+      <limit effort="${steering_effort}" velocity="6.28"  lower="-2.1" upper="2.1" />
       <dynamics damping="${steering_damping}" friction="${steering_friction}" />
     </joint>
@@ -283,5 +290,5 @@
       <axis
         xyz="0 0 -1" />
-      <limit effort="5" velocity="6.28"  lower="-2.1" upper="2.1" />
+      <limit effort="${steering_effort}" velocity="6.28"  lower="-2.1" upper="2.1" />
       <dynamics damping="${steering_damping}" friction="${steering_friction}" />
     </joint>
@@ -343,5 +350,5 @@
       <child link="${prefix}rr_steering_wheel_link"/>
       <axis xyz="0 0 -1" rpy="0 0 0" />
-      <limit effort="5" velocity="6.28"  lower="-2.1" upper="2.1" />
+      <limit effort="${steering_effort}" velocity="6.28"  lower="-2.1" upper="2.1" />
       <dynamics damping="${steering_damping}" friction="${steering_friction}" />
     </joint>

File: ranger_xarm6_description/robots/ranger_xarm6.urdf.xacro (robot description, xacro)
@@ -40,4 +40,9 @@
        See ranger_xarm6.launch.py, sim:=false path. -->
   <xacro:arg name="ros2_control_plugin" default="gz_ros2_control/GazeboSimSystem" />
+  <!-- Sim only: how the base moves. 'physics': gz_ros2_control drives the
+       4 steering joints (position) and 4 wheels (velocity), as
+       ranger_sim_base.py commands them from cmd_vel; 'kinematic': they're
+       passive and base_pose_publisher.py teleports the model. -->
+  <xacro:arg name="sim_base_drive" default="physics" />
   <xacro:arg name="robot_ip" default="" />
   <!-- ====================================================================
@@ -89,5 +94,6 @@
   <!-- Base: Ranger Mini 3.0 -->
   <xacro:include filename="$(find ranger_mini_v3_description)/urdf/ranger_mini_v3.xacro" />
-  <xacro:ranger_mini_v3 prefix="$(arg prefix)" />
+  <xacro:ranger_mini_v3 prefix="$(arg prefix)"
+    driven="${'$(arg ros2_control_plugin)' == 'gz_ros2_control/GazeboSimSystem' and '$(arg sim_base_drive)' == 'physics'}" />
   <!-- Arm: xArm6, mounted on the base via the placeholder FT above.
        model1300="true": this unit is the F/T-sensor-equipped "XI1300"
@@ -678,4 +684,15 @@
       <plugin filename="libgz-sim-sensors-system.so" name="gz::sim::systems::Sensors">
         <render_engine>ogre2</render_engine>
+      </plugin>
+    </gazebo>
+    <!-- The base's true motion (world pose, and body twist from it), on
+         /model/<entity>/odometry: ranger_sim_base.py publishes it as the
+         ground-truth odom -> base_link TF and ground_truth/odom. -->
+    <gazebo>
+      <plugin filename="gz-sim-odometry-publisher-system" name="gz::sim::systems::OdometryPublisher">
+        <odom_frame>odom</odom_frame>
+        <robot_base_frame>base_link</robot_base_frame>
+        <odom_publish_frequency>100</odom_publish_frequency>
+        <dimensions>3</dimensions>
       </plugin>
     </gazebo>
@@ -1266,8 +1283,9 @@
     <xacro:usb_camera_sensor_tags name="$(arg prefix)right_camera" />
   </xacro:if>
-  <!-- State-only ros2_control interface for the base's 4 steering + 4 wheel
-       joints (see ranger_mini_v3.xacro's own header comment: they're left
-       passive, no command interface / drive plugin; driving the base is
-       still separate follow-up work, unchanged by this). Without any
+  <!-- ros2_control interface for the base's 4 steering + 4 wheel joints.
+       sim_base_drive physics: steering position + wheel velocity commands
+       (steering_position_controller, wheel_velocity_controller, from
+       ranger_sim_base.py). kinematic: state only, the joints passive (the
+       base is teleported), as described below. Without any
        ros2_control interface, nothing ever published these joints' state,
        so robot_state_publisher had no value for them and couldn't compute
@@ -1290,18 +1308,23 @@
         <plugin>gz_ros2_control/GazeboSimSystem</plugin>
       </hardware>
-      <xacro:macro name="_passive_wheel_joint" params="name">
+      <!-- command: '' (state only), 'position' (steering) or 'velocity'
+           (wheels): commanded only with sim_base_drive physics. -->
+      <xacro:macro name="_passive_wheel_joint" params="name command:=''">
         <joint name="$(arg prefix)${name}">
+          <xacro:if value="${command and '$(arg sim_base_drive)' == 'physics'}">
+            <command_interface name="${command}"/>
+          </xacro:if>
           <state_interface name="position"/>
           <state_interface name="velocity"/>
         </joint>
       </xacro:macro>
-      <xacro:_passive_wheel_joint name="fl_steering_joint"/>
-      <xacro:_passive_wheel_joint name="fl_wheel"/>
-      <xacro:_passive_wheel_joint name="fr_steering_joint"/>
-      <xacro:_passive_wheel_joint name="fr_wheel"/>
-      <xacro:_passive_wheel_joint name="rl_steering_joint"/>
-      <xacro:_passive_wheel_joint name="rl_wheel"/>
-      <xacro:_passive_wheel_joint name="rr_steering_joint"/>
-      <xacro:_passive_wheel_joint name="rr_wheel"/>
+      <xacro:_passive_wheel_joint name="fl_steering_joint" command="position"/>
+      <xacro:_passive_wheel_joint name="fl_wheel" command="velocity"/>
+      <xacro:_passive_wheel_joint name="fr_steering_joint" command="position"/>
+      <xacro:_passive_wheel_joint name="fr_wheel" command="velocity"/>
+      <xacro:_passive_wheel_joint name="rl_steering_joint" command="position"/>
+      <xacro:_passive_wheel_joint name="rl_wheel" command="velocity"/>
+      <xacro:_passive_wheel_joint name="rr_steering_joint" command="position"/>
+      <xacro:_passive_wheel_joint name="rr_wheel" command="velocity"/>
       <!-- HiPNUC IMU state interface (see hipnuc_imu_sensor's <gazebo>
            block, below): purely to stop gz_ros2_control's GazeboSimSystem
